File: RightShift.sch (KiCad schematic (older format))
At the start: 9 parts

Commit message: Assign footprints, along with placeholders for mx
Parts:
- D57, D58, D59: renamed from D?; footprint (none) -> Diodes_SMD:D_SOD-123
- RS1, RS2, RS3, RS4, RS5, RS6: footprint (none) -> MX_Alps_Hybrid:MX-1U
Changed lines of the file:
@@
 F 0 "RS1" H 2675 2475 60  0000 C CNN
 F 1 "MX-1U" H 2675 2400 20  0000 C CNN
-F 2 "" H 2650 2325 60  0001 C CNN
+F 2 "MX_Alps_Hybrid:MX-1U" H 2650 2325 60  0001 C CNN
 F 3 "" H 2650 2325 60  0001 C CNN
 	1    2675 2350
@@
 $EndComp
 $Comp
-L D_Small D?
+L D_Small D57
 U 1 1 5A6855BE
 P 2575 2625
-F 0 "D?" H 2525 2705 50  0000 L CNN
+F 0 "D57" H 2525 2705 50  0000 L CNN
 F 1 "D_Small" H 2425 2545 50  0000 L CNN
-F 2 "" V 2575 2625 50  0001 C CNN
+F 2 "Diodes_SMD:D_SOD-123" V 2575 2625 50  0001 C CNN
 F 3 "" V 2575 2625 50  0001 C CNN
 	1    2575 2625
@@
 F 0 "RS5" H 3125 2475 60  0000 C CNN
 F 1 "MX-1U" H 3125 2400 20  0000 C CNN
-F 2 "" H 3100 2325 60  0001 C CNN
+F 2 "MX_Alps_Hybrid:MX-1U" H 3100 2325 60  0001 C CNN
 F 3 "" H 3100 2325 60  0001 C CNN
 	1    3125 2350
@@
 $EndComp
 $Comp
-L D_Small D?
+L D_Small D58
 U 1 1 5A6855CD
 P 3025 2625
-F 0 "D?" H 2975 2705 50  0000 L CNN
+F 0 "D58" H 2975 2705 50  0000 L CNN
 F 1 "D_Small" H 2875 2545 50  0000 L CNN
-F 2 "" V 3025 2625 50  0001 C CNN
+F 2 "Diodes_SMD:D_SOD-123" V 3025 2625 50  0001 C CNN
 F 3 "" V 3025 2625 50  0001 C CNN
 	1    3025 2625
@@
 F 0 "RS6" H 3575 2475 60  0000 C CNN
 F 1 "MX-1U" H 3575 2400 20  0000 C CNN
-F 2 "" H 3550 2325 60  0001 C CNN
+F 2 "MX_Alps_Hybrid:MX-1U" H 3550 2325 60  0001 C CNN
 F 3 "" H 3550 2325 60  0001 C CNN
 	1    3575 2350
@@
 $EndComp
 $Comp
-L D_Small D?
+L D_Small D59
 U 1 1 5A6855DC
 P 3475 2625
-F 0 "D?" H 3425 2705 50  0000 L CNN
+F 0 "D59" H 3425 2705 50  0000 L CNN
 F 1 "D_Small" H 3325 2545 50  0000 L CNN
-F 2 "" V 3475 2625 50  0001 C CNN
+F 2 "Diodes_SMD:D_SOD-123" V 3475 2625 50  0001 C CNN
 F 3 "" V 3475 2625 50  0001 C CNN
 	1    3475 2625
@@
 F 0 "RS3" H 2675 3100 60  0000 C CNN
 F 1 "MX-1U" H 2675 3025 20  0000 C CNN
-F 2 "" H 2650 2950 60  0001 C CNN
+F 2 "MX_Alps_Hybrid:MX-1U" H 2650 2950 60  0001 C CNN
 F 3 "" H 2650 2950 60  0001 C CNN
 	1    2675 2975
@@
 F 0 "RS4" H 3125 3100 60  0000 C CNN
 F 1 "MX-1U" H 3125 3025 20  0000 C CNN
-F 2 "" H 3100 2950 60  0001 C CNN
+F 2 "MX_Alps_Hybrid:MX-1U" H 3100 2950 60  0001 C CNN
 F 3 "" H 3100 2950 60  0001 C CNN
 	1    3125 2975
@@
 F 0 "RS2" H 3125 3625 60  0000 C CNN
 F 1 "MX-1U" H 3125 3550 20  0000 C CNN
-F 2 "" H 3100 3475 60  0001 C CNN
+F 2 "MX_Alps_Hybrid:MX-1U" H 3100 3475 60  0001 C CNN
 F 3 "" H 3100 3475 60  0001 C CNN
 	1    3125 3500

Commit message: Fix right shift sizes
Parts:
- RS2: value MX-1U -> MX-2.75U; footprint MX_Alps_Hybrid:MX-1U -> MX_Alps_Hybrid:MX-2.75U
- RS3, RS4: value MX-1U -> MX-1.75U; footprint MX_Alps_Hybrid:MX-1U -> MX_Alps_Hybrid:MX-1.75U
Changed lines of the file:
@@
 P 2675 2975
 F 0 "RS3" H 2675 3100 60  0000 C CNN
-F 1 "MX-1U" H 2675 3025 20  0000 C CNN
-F 2 "MX_Alps_Hybrid:MX-1U" H 2650 2950 60  0001 C CNN
+F 1 "MX-1.75U" H 2675 3025 20  0000 C CNN
+F 2 "MX_Alps_Hybrid:MX-1.75U" H 2650 2950 60  0001 C CNN
 F 3 "" H 2650 2950 60  0001 C CNN
 	1    2675 2975
@@
 P 3125 2975
 F 0 "RS4" H 3125 3100 60  0000 C CNN
-F 1 "MX-1U" H 3125 3025 20  0000 C CNN
-F 2 "MX_Alps_Hybrid:MX-1U" H 3100 2950 60  0001 C CNN
+F 1 "MX-1.75U" H 3125 3025 20  0000 C CNN
+F 2 "MX_Alps_Hybrid:MX-1.75U" H 3100 2950 60  0001 C CNN
 F 3 "" H 3100 2950 60  0001 C CNN
 	1    3125 2975
@@
 P 3125 3500
 F 0 "RS2" H 3125 3625 60  0000 C CNN
-F 1 "MX-1U" H 3125 3550 20  0000 C CNN
-F 2 "MX_Alps_Hybrid:MX-1U" H 3100 3475 60  0001 C CNN
+F 1 "MX-2.75U" H 3125 3550 20  0000 C CNN
+F 2 "MX_Alps_Hybrid:MX-2.75U" H 3100 3475 60  0001 C CNN
 F 3 "" H 3100 3475 60  0001 C CNN
 	1    3125 3500
