File: RightShift.sch (KiCad schematic (older format))
At the start: 9 parts

Commit message: Add basic row col to subsheets
Connections:
- net labels added: COL12, COL13, COL14, ROW3
- wire segments 3 -> 7
Changed lines of the file:
@@
 	1    0    0    -1
 $EndComp
+Wire Wire Line
+	3750 2325 3750 1925
+Wire Wire Line
+	3300 2300 3300 1925
+Wire Wire Line
+	2850 2325 2850 1925
+Text GLabel 2850 1925 1    60   Input ~ 0
+COL12
+Text GLabel 3300 1925 1    60   Input ~ 0
+COL13
+Text GLabel 3750 1925 1    60   Input ~ 0
+COL14
+Wire Wire Line
+	2125 2725 3475 2725
+Connection ~ 3025 2725
+Connection ~ 2575 2725
+Text GLabel 2125 2725 0    60   Input ~ 0
+ROW3
 $EndSCHEMATC

Commit message: Begin fixing rshift pinout
Parts:
- RS2: footprint MX_Alps_Hybrid:MX-2.75U -> MX_Alps_Hybrid:MX-2.75U-FLIPPED
Connections:
- wire segments 7 -> 12
Changed lines of the file:
@@
 $EndComp
 Wire Wire Line
-	2650 2525 2575 2525
+	2400 2525 2650 2525
 $Comp
 L MX-1U RS5
@@
 F 0 "RS2" H 3125 3625 60  0000 C CNN
 F 1 "MX-2.75U" H 3125 3550 20  0000 C CNN
-F 2 "MX_Alps_Hybrid:MX-2.75U" H 3100 3475 60  0001 C CNN
+F 2 "MX_Alps_Hybrid:MX-2.75U-FLIPPED" H 3100 3475 60  0001 C CNN
 F 3 "" H 3100 3475 60  0001 C CNN
 	1    3125 3500
@@
 	3300 2300 3300 1925
 Wire Wire Line
-	2850 2325 2850 1925
+	2850 1925 2850 2800
 Text GLabel 2850 1925 1    60   Input ~ 0
 COL12
@@
 Text GLabel 2125 2725 0    60   Input ~ 0
 ROW3
+Wire Wire Line
+	2850 2800 2650 2800
+Wire Wire Line
+	2650 2800 2650 3150
+Connection ~ 2850 2325
+Wire Wire Line
+	2850 2950 2850 2850
+Wire Wire Line
+	2850 2850 2400 2850
+Wire Wire Line
+	2400 2850 2400 2525
+Connection ~ 2575 2525
 $EndSCHEMATC

Commit message: Fully pinout rshift
Connections:
- wire segments 12 -> 20
Changed lines of the file:
@@
 $EndComp
 Wire Wire Line
-	3100 2525 3025 2525
+	2900 2525 3100 2525
 $Comp
 L MX-1U RS6
@@
 	3750 2325 3750 1925
 Wire Wire Line
-	3300 2300 3300 1925
+	3300 1925 3300 2650
 Wire Wire Line
 	2850 1925 2850 2800
@@
 	2400 2850 2400 2525
 Connection ~ 2575 2525
+Wire Wire Line
+	2900 2525 2900 3675
+Wire Wire Line
+	2900 3675 3100 3675
+Connection ~ 3025 2525
+Wire Wire Line
+	3300 2950 3300 2800
+Wire Wire Line
+	3300 2800 2900 2800
+Connection ~ 2900 2800
+Wire Wire Line
+	3300 2650 3350 2650
+Wire Wire Line
+	3350 2650 3350 3475
+Wire Wire Line
+	3350 3150 3100 3150
+Connection ~ 3300 2325
+Wire Wire Line
+	3350 3475 3300 3475
+Connection ~ 3350 3150
 $EndSCHEMATC

Commit message: Swap footprints for No-LED counterparts
Parts:
- RS1, RS5, RS6: footprint MX_Alps_Hybrid:MX-1U -> MX_Alps_Hybrid:MX-1U-NoLED
- RS2: footprint MX_Alps_Hybrid:MX-2.75U-FLIPPED -> MX_Alps_Hybrid:MX-2.75U-NoLED
- RS3, RS4: footprint MX_Alps_Hybrid:MX-1.75U -> MX_Alps_Hybrid:MX-1.75U-NoLED
Changed lines of the file:
@@
 F 0 "RS1" H 2675 2475 60  0000 C CNN
 F 1 "MX-1U" H 2675 2400 20  0000 C CNN
-F 2 "MX_Alps_Hybrid:MX-1U" H 2650 2325 60  0001 C CNN
+F 2 "MX_Alps_Hybrid:MX-1U-NoLED" H 2650 2325 60  0001 C CNN
 F 3 "" H 2650 2325 60  0001 C CNN
 	1    2675 2350
@@
 F 0 "RS5" H 3125 2475 60  0000 C CNN
 F 1 "MX-1U" H 3125 2400 20  0000 C CNN
-F 2 "MX_Alps_Hybrid:MX-1U" H 3100 2325 60  0001 C CNN
+F 2 "MX_Alps_Hybrid:MX-1U-NoLED" H 3100 2325 60  0001 C CNN
 F 3 "" H 3100 2325 60  0001 C CNN
 	1    3125 2350
@@
 F 0 "RS6" H 3575 2475 60  0000 C CNN
 F 1 "MX-1U" H 3575 2400 20  0000 C CNN
-F 2 "MX_Alps_Hybrid:MX-1U" H 3550 2325 60  0001 C CNN
+F 2 "MX_Alps_Hybrid:MX-1U-NoLED" H 3550 2325 60  0001 C CNN
 F 3 "" H 3550 2325 60  0001 C CNN
 	1    3575 2350
@@
 F 0 "RS3" H 2675 3100 60  0000 C CNN
 F 1 "MX-1.75U" H 2675 3025 20  0000 C CNN
-F 2 "MX_Alps_Hybrid:MX-1.75U" H 2650 2950 60  0001 C CNN
+F 2 "MX_Alps_Hybrid:MX-1.75U-NoLED" H 2650 2950 60  0001 C CNN
 F 3 "" H 2650 2950 60  0001 C CNN
 	1    2675 2975
@@
 F 0 "RS4" H 3125 3100 60  0000 C CNN
 F 1 "MX-1.75U" H 3125 3025 20  0000 C CNN
-F 2 "MX_Alps_Hybrid:MX-1.75U" H 3100 2950 60  0001 C CNN
+F 2 "MX_Alps_Hybrid:MX-1.75U-NoLED" H 3100 2950 60  0001 C CNN
 F 3 "" H 3100 2950 60  0001 C CNN
 	1    3125 2975
@@
 F 0 "RS2" H 3125 3625 60  0000 C CNN
 F 1 "MX-2.75U" H 3125 3550 20  0000 C CNN
-F 2 "MX_Alps_Hybrid:MX-2.75U-FLIPPED" H 3100 3475 60  0001 C CNN
+F 2 "MX_Alps_Hybrid:MX-2.75U-NoLED" H 3100 3475 60  0001 C CNN
 F 3 "" H 3100 3475 60  0001 C CNN
 	1    3125 3500

Commit message: Revert LED structure
Parts:
- RS1, RS5, RS6: footprint MX_Alps_Hybrid:MX-1U-NoLED -> MX_Alps_Hybrid:MX-1U
- RS2: footprint MX_Alps_Hybrid:MX-2.75U-NoLED -> MX_Alps_Hybrid:MX-2.75U
- RS3, RS4: footprint MX_Alps_Hybrid:MX-1.75U-NoLED -> MX_Alps_Hybrid:MX-1.75U
Changed lines of the file:
@@
 F 0 "RS1" H 2675 2475 60  0000 C CNN
 F 1 "MX-1U" H 2675 2400 20  0000 C CNN
-F 2 "MX_Alps_Hybrid:MX-1U-NoLED" H 2650 2325 60  0001 C CNN
+F 2 "MX_Alps_Hybrid:MX-1U" H 2650 2325 60  0001 C CNN
 F 3 "" H 2650 2325 60  0001 C CNN
 	1    2675 2350
@@
 F 0 "RS5" H 3125 2475 60  0000 C CNN
 F 1 "MX-1U" H 3125 2400 20  0000 C CNN
-F 2 "MX_Alps_Hybrid:MX-1U-NoLED" H 3100 2325 60  0001 C CNN
+F 2 "MX_Alps_Hybrid:MX-1U" H 3100 2325 60  0001 C CNN
 F 3 "" H 3100 2325 60  0001 C CNN
 	1    3125 2350
@@
 F 0 "RS6" H 3575 2475 60  0000 C CNN
 F 1 "MX-1U" H 3575 2400 20  0000 C CNN
-F 2 "MX_Alps_Hybrid:MX-1U-NoLED" H 3550 2325 60  0001 C CNN
+F 2 "MX_Alps_Hybrid:MX-1U" H 3550 2325 60  0001 C CNN
 F 3 "" H 3550 2325 60  0001 C CNN
 	1    3575 2350
@@
 F 0 "RS3" H 2675 3100 60  0000 C CNN
 F 1 "MX-1.75U" H 2675 3025 20  0000 C CNN
-F 2 "MX_Alps_Hybrid:MX-1.75U-NoLED" H 2650 2950 60  0001 C CNN
+F 2 "MX_Alps_Hybrid:MX-1.75U" H 2650 2950 60  0001 C CNN
 F 3 "" H 2650 2950 60  0001 C CNN
 	1    2675 2975
@@
 F 0 "RS4" H 3125 3100 60  0000 C CNN
 F 1 "MX-1.75U" H 3125 3025 20  0000 C CNN
-F 2 "MX_Alps_Hybrid:MX-1.75U-NoLED" H 3100 2950 60  0001 C CNN
+F 2 "MX_Alps_Hybrid:MX-1.75U" H 3100 2950 60  0001 C CNN
 F 3 "" H 3100 2950 60  0001 C CNN
 	1    3125 2975
@@
 F 0 "RS2" H 3125 3625 60  0000 C CNN
 F 1 "MX-2.75U" H 3125 3550 20  0000 C CNN
-F 2 "MX_Alps_Hybrid:MX-2.75U-NoLED" H 3100 3475 60  0001 C CNN
+F 2 "MX_Alps_Hybrid:MX-2.75U" H 3100 3475 60  0001 C CNN
 F 3 "" H 3100 3475 60  0001 C CNN
 	1    3125 3500
