File: RightShift.sch (KiCad schematic (older format))
At the start: 9 parts

Commit message: Wire LED rows
Connections:
- net LED-SW2: now reaches RS1.4 (LEDGND)
- net LED-SW2: now also RS5.4 (LEDGND), RS6.4 (LEDGND)
Changed lines of the file:
@@
 	3350 3475 3300 3475
 Connection ~ 3350 3150
+Text GLabel 2150 2475 0    60   Input ~ 0
+LED-SW2
+Wire Wire Line
+	2150 2475 3600 2475
+Connection ~ 2700 2475
+Connection ~ 3150 2475
 $EndSCHEMATC

Commit message: Begin routing
Connections:
- net LED-CS13: now reaches RS1.3 (LED)
- net LED-CS14: now reaches RS5.3 (LED)
- net LED-CS15: now reaches RS6.3 (LED)
Changed lines of the file:
@@
 Connection ~ 2700 2475
 Connection ~ 3150 2475
+Wire Wire Line
+	3700 2375 3700 1575
+Text GLabel 3700 1575 1    60   Input ~ 0
+LED-CS15
+Wire Wire Line
+	3250 2375 3250 1575
+Text GLabel 3250 1575 1    60   Input ~ 0
+LED-CS14
+Wire Wire Line
+	2800 2375 2800 1575
+Text GLabel 2800 1575 1    60   Input ~ 0
+LED-CS13
 $EndSCHEMATC

Commit message: Fix spacebar LED
Parts:
- RS2: footprint MX_Alps_Hybrid:MX-2.75U -> MX_Alps_Hybrid:MX-2.75U-FLIPPED
Connections:
- net LED-CS13: now also RS3.3 (LED)
- net LED-CS14: now also RS2.3 (LED), RS4.3 (LED)
- net LED-SW2: now also RS2.4 (LEDGND), RS3.4 (LEDGND), RS4.4 (LEDGND)
Changed lines of the file:
@@
 F 0 "RS2" H 3125 3625 60  0000 C CNN
 F 1 "MX-2.75U" H 3125 3550 20  0000 C CNN
-F 2 "MX_Alps_Hybrid:MX-2.75U" H 3100 3475 60  0001 C CNN
+F 2 "MX_Alps_Hybrid:MX-2.75U-FLIPPED" H 3100 3475 60  0001 C CNN
 F 3 "" H 3100 3475 60  0001 C CNN
 	1    3125 3500
@@
 LED-CS15
 Wire Wire Line
-	3250 2375 3250 1575
+	3250 1575 3250 3525
 Text GLabel 3250 1575 1    60   Input ~ 0
 LED-CS14
 Wire Wire Line
-	2800 2375 2800 1575
+	2800 1575 2800 3000
 Text GLabel 2800 1575 1    60   Input ~ 0
 LED-CS13
+Connection ~ 2800 2375
+Wire Wire Line
+	2700 3100 2700 2475
+Connection ~ 3250 2375
+Connection ~ 3250 3000
+Wire Wire Line
+	3150 2475 3150 3625
+Connection ~ 3150 3100
 $EndSCHEMATC
