File: VoyagerII.kicad_pcb (KiCad board)
At the start: 2 copper layers, 285 x 94.6 mm, 270 parts, among them P1 TC2030-IDC, SW1 SW_PUSH, U1 ATXMEGA32A4U-AU, U2 MCP1700T-3002E/TT, U3 STF202-22T1G, U4 IS31FL3731-SALS2

Commit message: Route cols
Routing:
- net COL12: track 36.1 -> 111.9 mm, vias 0 -> 1
- net COL13: track 35.4 -> 110.7 mm, vias 0 -> 1
- net COL11: track 39.0 -> 114.1 mm, vias 0 -> 1
- net COL14: track 42.7 -> 99.7 mm, vias 0 -> 1
- net COL4: track 23.0 -> 70.3 mm, vias 0 -> 1
- net COL9: track 41.0 -> 87.2 mm, vias 0 -> 2
- net COL3: track 34.7 -> 80.8 mm, vias 0 -> 1
- net COL10: track 37.9 -> 84.1 mm, vias 0 -> 1
- net COL5: track 38.6 -> 84.7 mm, vias 0 -> 1
- net COL2: track 33.1 -> 79.2 mm, vias 0 -> 1
- net COL8: track 43.9 -> 90.0 mm, vias 0 -> 1
- net COL7: track 45.8 -> 91.8 mm, vias 0 -> 1
- net COL6: track 53.8 -> 99.8 mm, vias 0 -> 1
- net Net-(D58-Pad2): track 0.00 -> 21.2 mm
- net Net-(D43-Pad2): track 0.00 -> 19.9 mm
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- added copper zone on F.Cu, net GND

Commit message: Route two rows
Routing:
- net ROW1: track 0.00 -> 267.1 mm, vias 0 -> 4
- net ROW0: track 8.18 -> 225.6 mm
- net COL14: track 99.7 -> 144.7 mm, vias 1 -> 2
- net Net-(D29-Pad2): track 0.00 -> 28.6 mm, vias 0 -> 1
- net COL10: track 84.1 -> 103.1 mm
- net Net-(D59-Pad2): track 0.00 -> 13.8 mm
- net Net-(D16-Pad2): track 0.00 -> 12.8 mm
- net Net-(D25-Pad2): track 0.00 -> 6.02 mm
- net Net-(D20-Pad2): track 0.00 -> 6.02 mm
- net Net-(D19-Pad2): track 0.00 -> 6.02 mm
- net Net-(D17-Pad2): track 0.00 -> 6.02 mm
- net Net-(D24-Pad2): track 0.00 -> 6.02 mm
- net Net-(D28-Pad2): track 0.00 -> 6.02 mm
- net Net-(D27-Pad2): track 0.00 -> 6.02 mm
- net Net-(D23-Pad2): track 0.00 -> 6.02 mm
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
Commit message: Route most of matrix
Routing:
- net ROW2: track 0.00 -> 281.2 mm, vias 0 -> 4
- net ROW4: track 0.00 -> 58.8 mm
- net COL0: track 44.3 -> 97.0 mm
- net Net-(D71-Pad2): track 0.00 -> 37.9 mm
- net Net-(D44-Pad2): track 0.00 -> 28.6 mm
- net COL2: track 79.2 -> 104.8 mm, vias 1 -> 2
- net COL1: track 67.9 -> 88.9 mm
- net Net-(D70-Pad2): track 0.00 -> 20.6 mm
- net Net-(D57-Pad2): track 0.00 -> 18.8 mm
- net Net-(D55-Pad2): track 0.00 -> 18.3 mm
- net Net-(D30-Pad2): track 0.00 -> 15.2 mm
- net Net-(D48-Pad2): track 0.00 -> 12.6 mm
- net Net-(D33-Pad2): track 0.00 -> 12.6 mm
- net Net-(D35-Pad2): track 0.00 -> 12.6 mm
- net COL6: track 99.8 -> 111.8 mm
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
Commit message: Connect all cols
Routing:
- net ROW3: track 0.00 -> 235.0 mm, vias 0 -> 6
- net COL14: track 145.0 -> 324.4 mm, vias 2 -> 4
- net COL13: track 114.9 -> 261.7 mm, vias 1 -> 3
- net COL12: track 121.5 -> 249.1 mm, vias 1 -> 3
- net COL11: track 114.1 -> 234.2 mm, vias 1 -> 4
- net COL10: track 103.1 -> 208.5 mm, vias 1 -> 3
- net COL9: track 87.2 -> 172.7 mm, vias 2 -> 4
- net COL0: track 97.0 -> 178.3 mm
- net COL8: track 90.0 -> 155.7 mm, vias 1 -> 3
- net COL1: track 88.9 -> 148.2 mm
- net +3V3: track 36.0 -> 89.8 mm, vias 0 -> 1
- net ROW4: track 58.8 -> 107.7 mm
- net COL4: track 70.3 -> 115.5 mm, vias 1 -> 2
- net COL7: track 91.8 -> 134.7 mm, vias 1 -> 2
- net COL3: track 80.8 -> 119.3 mm, vias 1 -> 2
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
Commit message: Continue routing
Routing:
- net ROW4: track 107.7 -> 193.2 mm, vias 0 -> 4
- net ROW1: track 267.1 -> 324.1 mm, vias 4 -> 6
- net ROW2: track 281.2 -> 333.9 mm, vias 4 -> 6
- net ROW3: track 235.0 -> 255.7 mm, vias 6 -> 8
Changed lines of the file:
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@@
     (thickness 1.6)
     (drawings 13)
-    (tracks 2190)
+    (tracks 2258)
     (zones 0)
     (modules 270)
@@
   (segment (start 53.34 54.61) (end 53.34 66.1275) (width 0.254) (layer F.Cu) (net 15))
   (segment (start 53.34 66.1275) (end 59.4125 72.2) (width 0.254) (layer F.Cu) (net 15))
+  (segment (start 148.40175 78.613) (end 132.715 78.613) (width 0.254) (layer B.Cu) (net 21))
+  (segment (start 132.715 78.613) (end 132.58575 78.613) (width 0.254) (layer B.Cu) (net 21))
+  (segment (start 132.715 78.105) (end 132.715 78.613) (width 0.254) (layer B.Cu) (net 21))
+  (segment (start 137.16 109.601) (end 132.435599 104.876599) (width 0.254) (layer F.Cu) (net 21))
+  (segment (start 132.435599 104.876599) (end 132.435599 94.658687) (width 0.254) (layer F.Cu) (net 21))
+  (segment (start 132.715 94.379286) (end 132.715 78.105) (width 0.254) (layer F.Cu) (net 21))
+  (segment (start 132.435599 94.658687) (end 132.715 94.379286) (width 0.254) (layer F.Cu) (net 21))
+  (via (at 132.715 78.105) (size 0.6) (drill 0.4) (layers F.Cu B.Cu) (net 21))
+  (segment (start 137.16 111.029994) (end 137.16 109.601) (width 0.254) (layer F.Cu) (net 21))
+  (segment (start 134.81051 113.411) (end 134.81051 113.379484) (width 0.254) (layer F.Cu) (net 21))
+  (segment (start 134.81051 113.379484) (end 137.16 111.029994) (width 0.254) (layer F.Cu) (net 21))
+  (segment (start 134.81051 113.60149) (end 134.81051 113.411) (width 0.254) (layer F.Cu) (net 21))
+  (segment (start 134.81051 115.063638) (end 134.81051 113.60149) (width 0.254) (layer F.Cu) (net 21))
+  (segment (start 132.969 116.967) (end 134.747 115.189) (width 0.254) (layer F.Cu) (net 21))
+  (segment (start 134.747 115.189) (end 134.747 115.127148) (width 0.254) (layer F.Cu) (net 21))
+  (segment (start 134.747 115.127148) (end 134.81051 115.063638) (width 0.254) (layer F.Cu) (net 21))
+  (segment (start 132.969 118.11) (end 132.969 116.967) (width 0.254) (layer F.Cu) (net 21))
+  (segment (start 139.334 125.999) (end 132.969 119.634) (width 0.254) (layer B.Cu) (net 21))
+  (segment (start 132.969 119.634) (end 132.969 118.11) (width 0.254) (layer B.Cu) (net 21))
+  (via (at 132.969 118.11) (size 0.6) (drill 0.4) (layers F.Cu B.Cu) (net 21))
+  (segment (start 141.4785 125.999) (end 139.334 125.999) (width 0.254) (layer B.Cu) (net 21))
   (segment (start 71.882 82.677) (end 69.088 82.677) (width 0.254) (layer B.Cu) (net 21))
   (segment (start 69.088 82.677) (end 65.024 78.613) (width 0.254) (layer B.Cu) (net 21))
@@
   (segment (start 130.96875 77.85) (end 130.11475 77.85) (width 0.254) (layer B.Cu) (net 21))
   (segment (start 130.11475 77.85) (end 129.35175 78.613) (width 0.254) (layer B.Cu) (net 21))
-  (segment (start 148.40175 78.613) (end 132.58575 78.613) (width 0.254) (layer B.Cu) (net 21))
   (segment (start 132.58575 78.613) (end 131.82275 77.85) (width 0.254) (layer B.Cu) (net 21))
   (segment (start 131.82275 77.85) (end 130.96875 77.85) (width 0.254) (layer B.Cu) (net 21))
@@
   (segment (start 302.41875 78.554) (end 306.017875 82.153125) (width 0.254) (layer B.Cu) (net 21))
   (segment (start 306.017875 82.153125) (end 306.721875 82.153125) (width 0.254) (layer B.Cu) (net 21))
+  (segment (start 116.68125 135) (end 116.714 135) (width 0.254) (layer B.Cu) (net 22))
+  (segment (start 116.714 135) (end 117.856 133.858) (width 0.254) (layer B.Cu) (net 22))
+  (segment (start 123.063 128.651) (end 117.856 133.858) (width 0.254) (layer F.Cu) (net 22))
+  (via (at 117.856 133.858) (size 0.6) (drill 0.4) (layers F.Cu B.Cu) (net 22))
+  (segment (start 138.1265 128.651) (end 123.063 128.651) (width 0.254) (layer B.Cu) (net 22))
+  (via (at 123.063 128.651) (size 0.6) (drill 0.4) (layers F.Cu B.Cu) (net 22))
+  (segment (start 139.7785 129.299) (end 138.7745 129.299) (width 0.254) (layer B.Cu) (net 22))
+  (segment (start 138.7745 129.299) (end 138.1265 128.651) (width 0.254) (layer B.Cu) (net 22))
+  (segment (start 229.87 136.144) (end 230.757121 137.031121) (width 0.254) (layer B.Cu) (net 22))
+  (segment (start 230.757121 137.031121) (end 245.713407 137.031121) (width 0.254) (layer B.Cu) (net 22))
+  (segment (start 245.713407 137.031121) (end 247.019627 135.724901) (width 0.254) (layer B.Cu) (net 22))
+  (segment (start 253.214849 135.724901) (end 253.93975 135) (width 0.254) (layer B.Cu) (net 22))
+  (segment (start 253.93975 135) (end 254.79375 135) (width 0.254) (layer B.Cu) (net 22))
+  (segment (start 247.019627 135.724901) (end 253.214849 135.724901) (width 0.254) (layer B.Cu) (net 22))
+  (segment (start 229.362 136.144) (end 229.87 136.144) (width 0.254) (layer F.Cu) (net 22))
+  (via (at 229.87 136.144) (size 0.6) (drill 0.4) (layers F.Cu B.Cu) (net 22))
+  (segment (start 226.06 136.144) (end 229.362 136.144) (width 0.254) (layer F.Cu) (net 22))
+  (segment (start 209.423 136.144) (end 226.06 136.144) (width 0.254) (layer F.Cu) (net 22))
+  (segment (start 197.739 136.144) (end 209.423 136.144) (width 0.254) (layer F.Cu) (net 22))
+  (segment (start 197.64375 135) (end 197.64375 136.04875) (width 0.254) (layer B.Cu) (net 22))
+  (segment (start 197.64375 136.04875) (end 197.739 136.144) (width 0.254) (layer B.Cu) (net 22))
+  (via (at 197.739 136.144) (size 0.6) (drill 0.4) (layers F.Cu B.Cu) (net 22))
   (segment (start 94.48575 135.763) (end 115.06425 135.763) (width 0.254) (layer B.Cu) (net 22))
   (segment (start 115.06425 135.763) (end 115.82725 135) (width 0.254) (layer B.Cu) (net 22))
@@
   (segment (start 254.79375 135) (end 255.64775 135) (width 0.254) (layer B.Cu) (net 22))
   (segment (start 255.64775 135) (end 258.365625 135) (width 0.254) (layer B.Cu) (net 22))
+  (segment (start 139.7785 128.499) (end 138.692934 128.499) (width 0.254) (layer B.Cu) (net 23))
+  (segment (start 138.692934 128.499) (end 135.724901 125.530967) (width 0.254) (layer B.Cu) (net 23))
+  (segment (start 135.724901 125.530967) (end 135.724901 124.040901) (width 0.254) (layer B.Cu) (net 23))
+  (segment (start 135.724901 124.040901) (end 130.937 119.253) (width 0.254) (layer B.Cu) (net 23))
+  (segment (start 130.937 119.253) (end 129.921 119.253) (width 0.254) (layer B.Cu) (net 23))
+  (segment (start 129.921 117.729) (end 129.921 114.808) (width 0.254) (layer F.Cu) (net 23))
+  (segment (start 129.921 118.237) (end 129.921 117.729) (width 0.254) (layer F.Cu) (net 23))
+  (segment (start 129.921 117.729) (end 129.921 119.253) (width 0.254) (layer F.Cu) (net 23))
+  (via (at 129.921 119.253) (size 0.6) (drill 0.4) (layers F.Cu B.Cu) (net 23))
+  (segment (start 129.921 114.808) (end 129.921 115.807125) (width 0.254) (layer B.Cu) (net 23))
+  (segment (start 129.921 115.807125) (end 129.778125 115.95) (width 0.254) (layer B.Cu) (net 23))
+  (via (at 129.921 114.808) (size 0.6) (drill 0.4) (layers F.Cu B.Cu) (net 23))
   (segment (start 290.938875 116.713) (end 312.708 116.713) (width 0.254) (layer B.Cu) (net 23))
   (segment (start 312.708 116.713) (end 313.471 115.95) (width 0.254) (layer B.Cu) (net 23))
@@
   (segment (start 106.30225 115.95) (end 107.15625 115.95) (width 0.254) (layer B.Cu) (net 23))
   (segment (start 88.10625 115.95) (end 91.678125 115.95) (width 0.254) (layer B.Cu) (net 23))
+  (segment (start 139.7785 127.699) (end 139.7785 127.17) (width 0.254) (layer B.Cu) (net 24))
+  (segment (start 139.7785 127.17) (end 131.0995 118.491) (width 0.254) (layer B.Cu) (net 24))
+  (segment (start 131.0995 118.491) (end 123.761501 118.491) (width 0.254) (layer B.Cu) (net 24))
+  (segment (start 123.761501 118.491) (end 121.539 120.713501) (width 0.254) (layer B.Cu) (net 24))
+  (segment (start 121.539 120.713501) (end 117.152419 120.713501) (width 0.254) (layer B.Cu) (net 24))
+  (segment (start 117.152419 120.713501) (end 116.078 119.639082) (width 0.254) (layer B.Cu) (net 24))
+  (segment (start 116.078 119.639082) (end 116.078 117.983) (width 0.254) (layer B.Cu) (net 24))
+  (segment (start 116.68125 96.9) (end 118.11 96.9) (width 0.254) (layer B.Cu) (net 24))
+  (segment (start 118.11 96.9) (end 120.253125 96.9) (width 0.254) (layer B.Cu) (net 24))
+  (segment (start 118.11 97.536) (end 118.11 96.9) (width 0.254) (layer B.Cu) (net 24))
+  (segment (start 116.078 117.983) (end 116.078 113.061994) (width 0.254) (layer F.Cu) (net 24))
+  (segment (start 116.078 113.061994) (end 118.11 111.029994) (width 0.254) (layer F.Cu) (net 24))
+  (segment (start 118.11 111.029994) (end 118.11 97.536) (width 0.254) (layer F.Cu) (net 24))
+  (via (at 118.11 97.536) (size 0.6) (drill 0.4) (layers F.Cu B.Cu) (net 24))
+  (via (at 116.078 117.983) (size 0.6) (drill 0.4) (layers F.Cu B.Cu) (net 24))
+  (segment (start 121.870125 97.663) (end 135.263118 97.663) (width 0.254) (layer B.Cu) (net 24))
   (segment (start 319.0875 96.9) (end 315.975 96.9) (width 0.254) (layer B.Cu) (net 24))
   (segment (start 309.568849 96.069151) (end 307.975 97.663) (width 0.254) (layer B.Cu) (net 24))
@@
   (segment (start 135.763 97.282) (end 139.827 97.282) (width 0.254) (layer F.Cu) (net 24))
   (via (at 139.827 97.282) (size 0.6) (drill 0.4) (layers F.Cu B.Cu) (net 24))
-  (segment (start 121.870125 97.663) (end 135.263118 97.663) (width 0.254) (layer B.Cu) (net 24))
   (segment (start 135.263118 97.663) (end 135.644118 97.282) (width 0.254) (layer B.Cu) (net 24))
   (segment (start 135.644118 97.282) (end 135.763 97.282) (width 0.254) (layer B.Cu) (net 24))
@@
   (segment (start 120.253125 96.9) (end 121.107125 96.9) (width 0.254) (layer B.Cu) (net 24))
   (segment (start 121.107125 96.9) (end 121.870125 97.663) (width 0.254) (layer B.Cu) (net 24))
-  (segment (start 116.68125 96.9) (end 120.253125 96.9) (width 0.254) (layer B.Cu) (net 24))
   (segment (start 99.24825 97.663) (end 115.06425 97.663) (width 0.254) (layer B.Cu) (net 24))
   (segment (start 115.06425 97.663) (end 115.82725 96.9) (width 0.254) (layer B.Cu) (net 24))

Commit message: Progress save
Routing:
- net PDI_CLK: track 25.1 -> 131.6 mm, vias 1 -> 2
- net ROW0: track 225.6 -> 302.3 mm, vias 0 -> 2
- net COL5: track 84.7 -> 112.8 mm, vias 1 -> 2
- net COL6: track 111.8 -> 112.6 mm
- net COL9: track 172.7 -> 173.2 mm

Commit message: Connect all
Hooray!
Routing:
- net GND: track 87.8 -> 926.6 mm, vias 5 -> 22
- net +5V: track 14.2 -> 842.9 mm, vias 0 -> 22
- net Net-(LED7-Pad2): track 0.00 -> 84.4 mm, vias 0 -> 2
- net ROW4: track 193.2 -> 269.5 mm, vias 4 -> 6
- net Net-(LED10-Pad4): track 0.00 -> 62.4 mm, vias 0 -> 2
- net Net-(LED4-Pad2): track 0.00 -> 53.8 mm
- net Net-(LED2-Pad2): track 0.00 -> 53.8 mm, vias 0 -> 2
- net Net-(LED11-Pad2): track 0.00 -> 53.8 mm
- net Net-(LED11-Pad4): track 0.00 -> 53.8 mm
- net Net-(LED6-Pad2): track 0.00 -> 52.4 mm
- net Net-(LED5-Pad2): track 0.00 -> 48.0 mm
- net Net-(LED3-Pad2): track 0.00 -> 47.3 mm, vias 0 -> 2
- net Net-(LED10-Pad2): track 0.00 -> 45.0 mm
- net Net-(LED1-Pad2): track 0.00 -> 42.5 mm, vias 0 -> 2
- net ROW0: track 302.3 -> 337.5 mm, vias 2 -> 4
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- removed copper zone on F.Cu, net GND

Commit message: Add logic schem module
Routing:
- net GND: track 926.6 -> 930.1 mm, vias 22 -> 23
- added copper zone on B.Cu, net GND
- added copper zone on F.Cu, net GND
Changed lines of the file:
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@@
     (thickness 1.6)
     (drawings 13)
-    (tracks 3011)
+    (tracks 3014)
     (zones 0)
     (modules 270)
@@
   (segment (start 153.188 131.699) (end 152.3095 131.699) (width 0.381) (layer B.Cu) (net 1))
   (segment (start 152.3095 131.699) (end 151.1785 131.699) (width 0.381) (layer B.Cu) (net 1))
+  (segment (start 67.8 54.25225) (end 67.8 52.321875) (width 0.381) (layer B.Cu) (net 2))
+  (segment (start 67.8 52.321875) (end 66.675 51.196875) (width 0.381) (layer B.Cu) (net 2))
+  (via (at 66.675 51.196875) (size 0.6) (drill 0.4) (layers F.Cu B.Cu) (net 2))
   (segment (start 164.2875 68.325) (end 165.5685 68.325) (width 0.381) (layer B.Cu) (net 2))
   (segment (start 165.5685 68.325) (end 166.713001 69.469501) (width 0.381) (layer B.Cu) (net 2))
@@
   (segment (start 166.18 123.256) (end 166.004 123.256) (width 0.254) (layer B.Cu) (net 144))
   (segment (start 166.004 123.256) (end 165.1 123.256) (width 0.254) (layer B.Cu) (net 144))
+  (zone (net 2) (net_name GND) (layer B.Cu) (hatch edge 0.508)
+    (connect_pads (clearance 0.381))
+    (min_thickness 0.254)
+    (fill yes (arc_segments 16) (thermal_gap 0.508) (thermal_bridge_width 0.508))
+    (polygon
+      (pts
+        (xy 47.625 47.625) (xy 59.53125 47.625) (xy 59.53125 57.15) (xy 72.628125 57.15) (xy 72.628125 47.625)
+        (xy 333.375 47.625) (xy 333.375 142.875) (xy 158.353125 142.875) (xy 158.353125 119.0625) (xy 126.20625 119.0625)
+        (xy 126.20625 142.875) (xy 47.625 142.875)
+      )
+    )
+  )
+  (zone (net 2) (net_name GND) (layer B.Cu) (hatch edge 0.508)
+    (connect_pads (clearance 0.381))
+    (min_thickness 0.254)
+    (fill yes (arc_segments 16) (thermal_gap 0.508) (thermal_bridge_width 0.508))
+    (polygon
+      (pts
+        (xy 60.721875 47.625) (xy 71.4375 47.625) (xy 71.4375 55.959375) (xy 60.721875 55.959375)
+      )
+    )
+  )
+  (zone (net 2) (net_name GND) (layer F.Cu) (hatch edge 0.508)
+    (connect_pads (clearance 0.381))
+    (min_thickness 0.254)
+    (fill yes (arc_segments 16) (thermal_gap 0.508) (thermal_bridge_width 0.508))
+    (polygon
+      (pts
+        (xy 47.625 47.625) (xy 59.53125 47.625) (xy 59.53125 57.15) (xy 72.628125 57.15) (xy 72.628125 47.625)
+        (xy 333.375 47.625) (xy 333.375 142.875) (xy 158.353125 142.875) (xy 158.353125 119.0625) (xy 126.20625 119.0625)
+        (xy 126.20625 142.875) (xy 47.625 142.875)
+      )
+    )
+  )
+  (zone (net 2) (net_name GND) (layer F.Cu) (hatch edge 0.508)
+    (connect_pads (clearance 0.381))
+    (min_thickness 0.254)
+    (fill yes (arc_segments 16) (thermal_gap 0.508) (thermal_bridge_width 0.508))
+    (polygon
+      (pts
+        (xy 60.721875 47.625) (xy 71.4375 47.625) (xy 71.4375 55.959375) (xy 60.721875 55.959375)
+      )
+    )
+  )
 )
