File: VoyagerII.kicad_pcb (KiCad board)
At the start: 2 copper layers, 285 x 95.1 mm, 197 parts, among them P1 TC2030-IDC, SW1 SW_PUSH, U1 ATXMEGA32A4U-AU, U2 MCP1700T-3002E/TT, U3 PRTR5V0U2X, U4 IS31FL3733, U5 74LVC1G34

Commit message: Continue routing
Parts:
- moved C3 0.63 mm to (137.8, 137.7)
- moved C4 0.52 mm to (154.1, 131.3)
- moved R1 0.13 mm to (154.1, 126.7)
Routing:
- net I2C+: track 0.00 -> 186.2 mm, vias 0 -> 4
- net I2C-: track 0.00 -> 184.4 mm, vias 0 -> 4
- net COL1: track 0.00 -> 144.2 mm
- net GND: track 100.8 -> 216.2 mm, vias 8 -> 14
- net COL0: track 86.9 -> 184.4 mm
- net +3V3: track 16.1 -> 97.5 mm, vias 0 -> 3
- net +5V: track 22.5 -> 86.2 mm
- net COL3: track 64.3 -> 111.0 mm, vias 0 -> 1
- net Net-(LED10-Pad2): track 0.00 -> 44.2 mm
- net COL4: track 64.3 -> 106.9 mm, vias 0 -> 1
- net PDI: track 0.00 -> 33.6 mm, vias 0 -> 1
- net COL2: track 64.3 -> 97.1 mm
- net PDI_CLK: track 3.71 -> 25.0 mm, vias 0 -> 1
- net Net-(D57-Pad2): track 0.00 -> 18.5 mm
- net Net-(D29-Pad2): track 0.00 -> 18.0 mm
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
Commit message: Fix spacebar LED
Parts:
- RS2: footprint MX_Alps_Hybrid:MX-2.75U -> MX_Alps_Hybrid:MX-2.75U-FLIPPED
Connections:
- RS2 pad 3: Net-(RS2-Pad3) -> LED-CS14
- RS2 pad 4: Net-(RS2-Pad4) -> LED-SW2
- RS3 pad 3: Net-(RS3-Pad3) -> LED-CS13
- RS3 pad 4: Net-(RS3-Pad4) -> LED-SW2
- RS4 pad 3: Net-(RS4-Pad3) -> LED-CS14
- RS4 pad 4: Net-(RS4-Pad4) -> LED-SW2
- SP1 pad 3: Net-(SP1-Pad3) -> LED-CS7
- U4 pad 49: GND -> (no net)
Routing:
- net LED-SW2: track 146.6 -> 208.1 mm
- net COL2: track 97.1 -> 134.9 mm, vias 0 -> 1
- net LED-CS14: track 51.4 -> 86.3 mm
- net GND: track 216.2 -> 248.6 mm, vias 14 -> 18
- net LED-CS7: track 216.0 -> 246.1 mm
- net ROW4: track 114.5 -> 144.0 mm, vias 0 -> 2
- net COL6: track 109.2 -> 136.3 mm
- net Net-(D58-Pad2): track 0.00 -> 23.0 mm, vias 0 -> 2
- net Net-(D59-Pad2): track 0.00 -> 16.1 mm
- net ROW0: track 225.1 -> 240.3 mm, vias 0 -> 1
- net ROW3: track 188.6 -> 202.7 mm, vias 4 -> 5
- net COL14: track 289.3 -> 302.8 mm
- net ROW1: track 264.3 -> 277.7 mm, vias 0 -> 1
- net ROW2: track 231.6 -> 244.7 mm, vias 0 -> 1
- net Net-(D62-Pad2): track 0.00 -> 10.6 mm
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
Commit message: Finish routing
Parts:
- moved D43 15.1 mm to (304.0, 95.2)
Routing:
- net GND: track 248.6 -> 2163.9 mm, vias 18 -> 59
- net +5V: track 86.2 -> 876.7 mm, vias 0 -> 14
- net LED-SW1: track 131.2 -> 342.6 mm, vias 0 -> 3
- net +3V3: track 97.5 -> 245.9 mm, vias 3 -> 4
- net ROW0: track 240.3 -> 374.8 mm, vias 1 -> 6
- net ROW4: track 144.0 -> 271.6 mm, vias 2 -> 4
- net PDI_CLK: track 25.0 -> 136.6 mm, vias 1 -> 2
- net LED-SW2: track 208.1 -> 312.6 mm, vias 0 -> 4
- net Net-(LED7-Pad2): track 0.00 -> 73.7 mm, vias 0 -> 2
- net ROW2: track 244.7 -> 315.8 mm, vias 1 -> 4
- net ROW3: track 202.7 -> 272.4 mm, vias 5 -> 6
- net Net-(LED10-Pad4): track 0.00 -> 61.3 mm, vias 0 -> 2
- net LED-CS13: track 86.9 -> 144.7 mm
- net LED-SW5: track 282.2 -> 339.3 mm, vias 0 -> 2
- net Net-(LED11-Pad4): track 0.00 -> 55.3 mm
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Other:
- board text removed: "Lo and Behold!"

Commit message: Finalize for error checking
Other:
- net class Default: clearance 0.254 -> 0.1778
- net class Power: clearance 0.254 -> 0.1778
- rule trace_clearance: 0.254 -> 0.1778
Changed lines of the file:
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@@
   (setup
     (last_trace_width 0.254)
-    (trace_clearance 0.254)
+    (trace_clearance 0.1778)
     (zone_clearance 0.381)
     (zone_45_only no)
@@
   (net 157 LED-CS14)
   (net_class Default "This is the default net class."
-    (clearance 0.254)
+    (clearance 0.1778)
     (trace_width 0.254)
     (via_dia 0.6)
@@
   )
   (net_class Power ""
-    (clearance 0.254)
+    (clearance 0.1778)
     (trace_width 0.381)
     (via_dia 0.6)

Commit message: Improve routing
Routing:
- net COL14: track 303.7 -> 301.8 mm
- net GND: track 2163.9 -> 2163.2 mm
Changed lines of the file:
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@@
     (links 666)
     (no_connects 0)
-    (area 28.932287 28.25625 334.554951 153.909376)
+    (area 28.932287 28.25625 334.478751 153.909376)
     (thickness 1.6)
     (drawings 41)
-    (tracks 3175)
+    (tracks 3177)
     (zones 0)
     (modules 197)
@@
     (clearance 0.127)
     (attr virtual)
-    (fp_text reference P1 (at -3.048 2.54 540) (layer B.SilkS)
+    (fp_text reference P1 (at 3.048 -2.794 540) (layer B.SilkS)
       (effects (font (size 0.75692 0.75692) (thickness 0.127)) (justify mirror))
     )
@@
     (effects (font (size 1 1) (thickness 0.15)) (justify mirror))
   )
-  (gr_text "CLK\n" (at 162.56 138.049) (layer B.SilkS)
+  (gr_text "CLK\n" (at 164.084 139.954) (layer B.SilkS)
     (effects (font (size 1 1) (thickness 0.15)) (justify mirror))
   )
-  (gr_text GND (at 162.306 135.509) (layer B.SilkS)
+  (gr_text GND (at 164.338 133.731) (layer B.SilkS)
     (effects (font (size 1 1) (thickness 0.15)) (justify mirror))
   )
@@
   (segment (start 292.484 100.454) (end 291.453 101.485) (width 0.2286) (layer B.Cu) (net 1))
   (segment (start 291.453 101.485) (end 290.703 101.485) (width 0.2286) (layer B.Cu) (net 1))
+  (segment (start 62.103 55.118) (end 63.754 55.118) (width 0.381) (layer F.Cu) (net 2))
+  (segment (start 63.754 55.118) (end 70.485 55.118) (width 0.381) (layer F.Cu) (net 2))
+  (segment (start 65.024 56.388) (end 63.754 55.118) (width 0.381) (layer F.Cu) (net 2))
+  (segment (start 65.024 59.944) (end 65.024 56.388) (width 0.381) (layer F.Cu) (net 2))
   (segment (start 311.912 128.905) (end 305.308 122.301) (width 0.381) (layer F.Cu) (net 2))
   (via (at 299.72 122.301) (size 0.6) (drill 0.4) (layers F.Cu B.Cu) (net 2))
@@
   (segment (start 68.58 59.944) (end 68.58 60.448) (width 0.381) (layer B.Cu) (net 2))
   (segment (start 68.58 60.448) (end 67.421 61.607) (width 0.381) (layer B.Cu) (net 2))
-  (segment (start 65.024 59.944) (end 65.024 58.039) (width 0.381) (layer F.Cu) (net 2))
-  (segment (start 65.024 58.039) (end 62.103 55.118) (width 0.381) (layer F.Cu) (net 2))
   (segment (start 69.4626 54.195) (end 69.562 54.195) (width 0.381) (layer B.Cu) (net 2))
   (segment (start 69.562 54.195) (end 70.485 55.118) (width 0.381) (layer B.Cu) (net 2))
-  (segment (start 62.103 55.118) (end 70.485 55.118) (width 0.381) (layer F.Cu) (net 2))
   (via (at 70.485 55.118) (size 0.6) (drill 0.4) (layers F.Cu B.Cu) (net 2))
   (segment (start 63.0126 54.195) (end 63.0126 54.2084) (width 0.381) (layer B.Cu) (net 2))
@@
   (segment (start 169.418 134.239) (end 170.561 134.239) (width 0.254) (layer B.Cu) (net 30))
   (segment (start 170.561 134.239) (end 171.323 135.001) (width 0.254) (layer B.Cu) (net 30))
+  (segment (start 318.516 129.032) (end 320.929 126.619) (width 0.254) (layer B.Cu) (net 33))
+  (segment (start 316.5875 129.35) (end 318.198 129.35) (width 0.254) (layer B.Cu) (net 33))
+  (segment (start 318.198 129.35) (end 318.516 129.032) (width 0.254) (layer B.Cu) (net 33))
   (segment (start 151.1785 132.499) (end 152.273 132.499) (width 0.254) (layer B.Cu) (net 33))
   (segment (start 152.273 132.499) (end 152.623001 132.849001) (width 0.254) (layer B.Cu) (net 33))
@@
   (segment (start 315.976 107.696) (end 320.04 111.76) (width 0.254) (layer B.Cu) (net 33))
   (segment (start 324.739 126.619) (end 321.056 126.619) (width 0.254) (layer B.Cu) (net 33))
-  (segment (start 315.2775 130.81) (end 316.738 130.81) (width 0.254) (layer B.Cu) (net 33))
-  (segment (start 316.738 130.81) (end 320.929 126.619) (width 0.254) (layer B.Cu) (net 33))
   (segment (start 320.929 126.619) (end 321.056 126.619) (width 0.254) (layer B.Cu) (net 33))
   (segment (start 326.39 128.27) (end 324.739 126.619) (width 0.254) (layer B.Cu) (net 33))
@@
   (segment (start 60.6425 86.512368) (end 63.577251 89.447119) (width 0.254) (layer F.Cu) (net 156))
   (segment (start 63.577251 89.447119) (end 63.577251 91.870749) (width 0.254) (layer F.Cu) (net 156))
+  (segment (start 296.38625 119.38) (end 297.78325 117.983) (width 0.254) (layer F.Cu) (net 157))
+  (segment (start 297.78325 117.983) (end 302.133 117.983) (width 0.254) (layer F.Cu) (net 157))
+  (segment (start 302.577501 118.427501) (end 303.53 119.38) (width 0.254) (layer F.Cu) (net 157))
+  (segment (start 302.133 117.983) (end 302.577501 118.427501) (width 0.254) (layer F.Cu) (net 157))
+  (segment (start 308.45125 118.032962) (end 308.45125 119.38) (width 0.254) (layer F.Cu) (net 157))
+  (segment (start 304.653949 118.046499) (end 307.327301 118.046499) (width 0.254) (layer F.Cu) (net 157))
+  (segment (start 304.482499 118.427501) (end 304.482499 118.217949) (width 0.254) (layer F.Cu) (net 157))
+  (segment (start 307.327301 118.046499) (end 307.498751 118.217949) (width 0.254) (layer F.Cu) (net 157))
+  (segment (start 307.498751 118.217949) (end 307.498751 118.427501) (width 0.254) (layer F.Cu) (net 157))
+  (segment (start 307.498751 118.427501) (end 308.45125 119.38) (width 0.254) (layer F.Cu) (net 157))
+  (segment (start 303.53 119.38) (end 304.482499 118.427501) (width 0.254) (layer F.Cu) (net 157))
+  (segment (start 304.482499 118.217949) (end 304.653949 118.046499) (width 0.254) (layer F.Cu) (net 157))
   (segment (start 304.038 95.331) (end 305.054 96.347) (width 0.254) (layer F.Cu) (net 157))
   (segment (start 305.054 96.347) (end 305.054 100.838) (width 0.254) (layer F.Cu) (net 157))
@@
   (segment (start 313.493151 109.277151) (end 313.493151 114.891313) (width 0.254) (layer F.Cu) (net 157))
   (segment (start 313.493151 114.891313) (end 312.687464 115.697) (width 0.254) (layer F.Cu) (net 157))
-  (segment (start 308.45125 118.032962) (end 308.45125 119.38) (width 0.254) (layer F.Cu) (net 157))
   (segment (start 312.687464 115.697) (end 310.787212 115.697) (width 0.254) (layer F.Cu) (net 157))
   (segment (start 310.787212 115.697) (end 308.45125 118.032962) (width 0.254) (layer F.Cu) (net 157))
@@
   (segment (start 297.307 85.217) (end 294.005 81.915) (width 0.254) (layer B.Cu) (net 157))
   (segment (start 301.244 96.012) (end 301.244 92.456) (width 0.254) (layer B.Cu) (net 157))
-  (segment (start 296.38625 119.38) (end 297.78325 117.983) (width 0.254) (layer F.Cu) (net 157))
-  (segment (start 297.78325 117.983) (end 302.133 117.983) (width 0.254) (layer F.Cu) (net 157))
-  (segment (start 302.133 117.983) (end 302.577501 118.427501) (width 0.254) (layer F.Cu) (net 157))
-  (segment (start 302.577501 118.427501) (end 303.53 119.38) (width 0.254) (layer F.Cu) (net 157))
-  (segment (start 303.53 119.38) (end 304.482499 118.427501) (width 0.254) (layer F.Cu) (net 157))
-  (segment (start 304.482499 118.427501) (end 304.482499 118.217949) (width 0.254) (layer F.Cu) (net 157))
-  (segment (start 307.498751 118.217949) (end 307.498751 118.427501) (width 0.254) (layer F.Cu) (net 157))
-  (segment (start 304.482499 118.217949) (end 304.653949 118.046499) (width 0.254) (layer F.Cu) (net 157))
-  (segment (start 307.327301 118.046499) (end 307.498751 118.217949) (width 0.254) (layer F.Cu) (net 157))
-  (segment (start 304.653949 118.046499) (end 307.327301 118.046499) (width 0.254) (layer F.Cu) (net 157))
-  (segment (start 307.498751 118.427501) (end 308.45125 119.38) (width 0.254) (layer F.Cu) (net 157))
   (segment (start 296.037 96.139) (end 296.037 96.647) (width 0.2286) (layer B.Cu) (net 157))
   (segment (start 295.602 95.704) (end 296.037 96.139) (width 0.2286) (layer B.Cu) (net 157))
@@
     (polygon
       (pts
-        (xy 60.706 47.498) (xy 60.706 55.88) (xy 71.374 55.88) (xy 71.374 47.498)
+        (xy 60.706 47.498) (xy 60.706 55.88) (xy 62.23 55.88) (xy 62.23 56.642) (xy 71.374 56.642)
+        (xy 71.374 55.88) (xy 71.374 47.498)
       )
     )

Commit message: Temporary save during trace cleanup
Routing:
- net COL0: track 186.3 -> 190.3 mm
- net GND: track 2163.2 -> 2162.8 mm, vias 59 -> 57

Commit message: Update fill and logo text
Parts:
- moved REF** 135.4 mm to (209.2, 133.3)

Commit message: Tune up routing
Parts:
- moved R2 0.96 mm to (286.8, 100.8)
Connections:
- U4 pad 46: Net-(U4-Pad46) -> +3V3
Routing:
- net GND: track 2162.8 -> 2208.0 mm, vias 57 -> 60
- net +3V3: track 245.9 -> 254.4 mm
- net Net-(R8-Pad1): track 12.1 -> 14.1 mm
- net LED-CS15: track 132.7 -> 133.4 mm
- net Net-(D62-Pad2): track 12.6 -> 13.3 mm
