File: RGB.sch (KiCad schematic (older format))
At the start: 26 parts, among them U5 74LVC1G34

Commit message: Revert LED structure
Parts:
- CRGB1, CRGB10, CRGB11, CRGB12, CRGB2, CRGB3, CRGB4, CRGB5, CRGB6, CRGB7, CRGB8, CRGB9: footprint Capacitors_SMD:C_0805 -> Capacitors_SMD:C_0603
- R5: footprint Resistors_SMD:R_0805 -> Resistors_SMD:R_0603
Changed lines of the file:
@@
 F 0 "CRGB1" H 5685 2420 50  0000 L CNN
 F 1 "0.1u" H 5685 2270 50  0000 L CNN
-F 2 "Capacitors_SMD:C_0805" H 5675 2350 50  0001 C CNN
+F 2 "Capacitors_SMD:C_0603" H 5675 2350 50  0001 C CNN
 F 3 "" H 5675 2350 50  0001 C CNN
 	1    5675 2350
@@
 F 0 "CRGB2" H 5960 2420 50  0000 L CNN
 F 1 "0.1u" H 5960 2270 50  0000 L CNN
-F 2 "Capacitors_SMD:C_0805" H 5950 2350 50  0001 C CNN
+F 2 "Capacitors_SMD:C_0603" H 5950 2350 50  0001 C CNN
 F 3 "" H 5950 2350 50  0001 C CNN
 	1    5950 2350
@@
 F 0 "CRGB3" H 6235 2420 50  0000 L CNN
 F 1 "0.1u" H 6235 2270 50  0000 L CNN
-F 2 "Capacitors_SMD:C_0805" H 6225 2350 50  0001 C CNN
+F 2 "Capacitors_SMD:C_0603" H 6225 2350 50  0001 C CNN
 F 3 "" H 6225 2350 50  0001 C CNN
 	1    6225 2350
@@
 F 0 "CRGB4" H 6510 2420 50  0000 L CNN
 F 1 "0.1u" H 6510 2270 50  0000 L CNN
-F 2 "Capacitors_SMD:C_0805" H 6500 2350 50  0001 C CNN
+F 2 "Capacitors_SMD:C_0603" H 6500 2350 50  0001 C CNN
 F 3 "" H 6500 2350 50  0001 C CNN
 	1    6500 2350
@@
 F 0 "CRGB5" H 6785 2420 50  0000 L CNN
 F 1 "0.1u" H 6785 2270 50  0000 L CNN
-F 2 "Capacitors_SMD:C_0805" H 6775 2350 50  0001 C CNN
+F 2 "Capacitors_SMD:C_0603" H 6775 2350 50  0001 C CNN
 F 3 "" H 6775 2350 50  0001 C CNN
 	1    6775 2350
@@
 F 0 "CRGB6" H 7060 2420 50  0000 L CNN
 F 1 "0.1u" H 7060 2270 50  0000 L CNN
-F 2 "Capacitors_SMD:C_0805" H 7050 2350 50  0001 C CNN
+F 2 "Capacitors_SMD:C_0603" H 7050 2350 50  0001 C CNN
 F 3 "" H 7050 2350 50  0001 C CNN
 	1    7050 2350
@@
 F 0 "CRGB7" H 5685 2745 50  0000 L CNN
 F 1 "0.1u" H 5685 2595 50  0000 L CNN
-F 2 "Capacitors_SMD:C_0805" H 5675 2675 50  0001 C CNN
+F 2 "Capacitors_SMD:C_0603" H 5675 2675 50  0001 C CNN
 F 3 "" H 5675 2675 50  0001 C CNN
 	1    5675 2675
@@
 F 0 "CRGB8" H 5960 2745 50  0000 L CNN
 F 1 "0.1u" H 5960 2595 50  0000 L CNN
-F 2 "Capacitors_SMD:C_0805" H 5950 2675 50  0001 C CNN
+F 2 "Capacitors_SMD:C_0603" H 5950 2675 50  0001 C CNN
 F 3 "" H 5950 2675 50  0001 C CNN
 	1    5950 2675
@@
 F 0 "CRGB9" H 6235 2745 50  0000 L CNN
 F 1 "0.1u" H 6235 2595 50  0000 L CNN
-F 2 "Capacitors_SMD:C_0805" H 6225 2675 50  0001 C CNN
+F 2 "Capacitors_SMD:C_0603" H 6225 2675 50  0001 C CNN
 F 3 "" H 6225 2675 50  0001 C CNN
 	1    6225 2675
@@
 F 0 "CRGB10" H 6510 2745 50  0000 L CNN
 F 1 "0.1u" H 6510 2595 50  0000 L CNN
-F 2 "Capacitors_SMD:C_0805" H 6500 2675 50  0001 C CNN
+F 2 "Capacitors_SMD:C_0603" H 6500 2675 50  0001 C CNN
 F 3 "" H 6500 2675 50  0001 C CNN
 	1    6500 2675
@@
 F 0 "CRGB11" H 6785 2745 50  0000 L CNN
 F 1 "0.1u" H 6785 2595 50  0000 L CNN
-F 2 "Capacitors_SMD:C_0805" H 6775 2675 50  0001 C CNN
+F 2 "Capacitors_SMD:C_0603" H 6775 2675 50  0001 C CNN
 F 3 "" H 6775 2675 50  0001 C CNN
 	1    6775 2675
@@
 F 0 "CRGB12" H 7060 2745 50  0000 L CNN
 F 1 "0.1u" H 7060 2595 50  0000 L CNN
-F 2 "Capacitors_SMD:C_0805" H 7050 2675 50  0001 C CNN
+F 2 "Capacitors_SMD:C_0603" H 7050 2675 50  0001 C CNN
 F 3 "" H 7050 2675 50  0001 C CNN
 	1    7050 2675
@@
 F 0 "R5" H 2805 1445 50  0000 L CNN
 F 1 "500" H 2805 1385 50  0000 L CNN
-F 2 "Resistors_SMD:R_0805" H 2775 1425 50  0001 C CNN
+F 2 "Resistors_SMD:R_0603" H 2775 1425 50  0001 C CNN
 F 3 "" H 2775 1425 50  0001 C CNN
 	1    2775 1425
