File: VoyagerII.sch (KiCad schematic (older format))
At the start: 29 parts, among them P1 TC2030-IDC, SW1 SW_PUSH, U1 ATXMEGA32A4U-AU, U2 MCP1700T-3002E/TT, U3 PRTR5V0U2X, U4 IS31FL3733

Commit message: Update netlist
Parts:
- U4: footprint (none) -> Housings_DFN_QFN:QFN-48-1EP_6x6mm_Pitch0.4mm
Changed lines of the file:
@@
 $EndComp
 $Comp
-L VCC #PWR20
+L VCC #PWR01
 U 1 1 5A6244BE
 P 9250 1325
-F 0 "#PWR20" H 9250 1175 50  0001 C CNN
+F 0 "#PWR01" H 9250 1175 50  0001 C CNN
 F 1 "VCC" H 9250 1475 50  0000 C CNN
 F 2 "" H 9250 1325 50  0001 C CNN
@@
 $EndComp
 $Comp
-L +5V #PWR23
+L +5V #PWR02
 U 1 1 5A6244DC
 P 9600 1275
-F 0 "#PWR23" H 9600 1125 50  0001 C CNN
+F 0 "#PWR02" H 9600 1125 50  0001 C CNN
 F 1 "+5V" H 9600 1415 50  0000 C CNN
 F 2 "" H 9600 1275 50  0001 C CNN
@@
 $EndComp
 $Comp
-L +5V #PWR7
+L +5V #PWR03
 U 1 1 5A624862
 P 3425 1300
-F 0 "#PWR7" H 3425 1150 50  0001 C CNN
+F 0 "#PWR03" H 3425 1150 50  0001 C CNN
 F 1 "+5V" H 3425 1440 50  0000 C CNN
 F 2 "" H 3425 1300 50  0001 C CNN
@@
 $EndComp
 $Comp
-L GND #PWR10
+L GND #PWR04
 U 1 1 5A6248B2
 P 3925 1600
-F 0 "#PWR10" H 3925 1350 50  0001 C CNN
+F 0 "#PWR04" H 3925 1350 50  0001 C CNN
 F 1 "GND" H 3925 1450 50  0000 C CNN
 F 2 "" H 3925 1600 50  0001 C CNN
@@
 $EndComp
 $Comp
-L GND #PWR11
+L GND #PWR05
 U 1 1 5A624D2D
 P 4300 1500
-F 0 "#PWR11" H 4300 1250 50  0001 C CNN
+F 0 "#PWR05" H 4300 1250 50  0001 C CNN
 F 1 "GND" H 4300 1350 50  0000 C CNN
 F 2 "" H 4300 1500 50  0001 C CNN
@@
 $EndComp
 $Comp
-L +3.3V #PWR6
+L +3.3V #PWR06
 U 1 1 5A625634
 P 2550 2300
-F 0 "#PWR6" H 2550 2150 50  0001 C CNN
+F 0 "#PWR06" H 2550 2150 50  0001 C CNN
 F 1 "+3.3V" H 2550 2440 50  0000 C CNN
 F 2 "" H 2550 2300 50  0000 C CNN
@@
 $EndComp
 $Comp
-L GND #PWR5
+L GND #PWR07
 U 1 1 5A625723
 P 1900 2500
-F 0 "#PWR5" H 1900 2250 50  0001 C CNN
+F 0 "#PWR07" H 1900 2250 50  0001 C CNN
 F 1 "GND" H 1900 2350 50  0000 C CNN
 F 2 "" H 1900 2500 50  0000 C CNN
@@
 PDI_CLK
 $Comp
-L GND #PWR4
+L GND #PWR08
 U 1 1 5A62606A
 P 1650 2625
-F 0 "#PWR4" H 1650 2375 50  0001 C CNN
+F 0 "#PWR08" H 1650 2375 50  0001 C CNN
 F 1 "GND" H 1650 2475 50  0000 C CNN
 F 2 "" H 1650 2625 50  0000 C CNN
@@
 PDI
 $Comp
-L +3.3V #PWR8
+L +3.3V #PWR09
 U 1 1 5A6265F5
 P 3575 2050
-F 0 "#PWR8" H 3575 1900 50  0001 C CNN
+F 0 "#PWR09" H 3575 1900 50  0001 C CNN
 F 1 "+3.3V" H 3575 2190 50  0000 C CNN
 F 2 "" H 3575 2050 50  0000 C CNN
@@
 $EndComp
 $Comp
-L GND #PWR9
+L GND #PWR010
 U 1 1 5A626934
 P 3825 4950
-F 0 "#PWR9" H 3825 4700 50  0001 C CNN
+F 0 "#PWR010" H 3825 4700 50  0001 C CNN
 F 1 "GND" H 3825 4800 50  0000 C CNN
 F 2 "" H 3825 4950 50  0000 C CNN
@@
 $EndComp
 $Comp
-L +3.3V #PWR1
+L +3.3V #PWR011
 U 1 1 5A627061
 P 725 3075
-F 0 "#PWR1" H 725 2925 50  0001 C CNN
+F 0 "#PWR011" H 725 2925 50  0001 C CNN
 F 1 "+3.3V" H 725 3215 50  0000 C CNN
 F 2 "" H 725 3075 50  0000 C CNN
@@
 $EndComp
 $Comp
-L GND #PWR2
+L GND #PWR012
 U 1 1 5A62709B
 P 725 3275
-F 0 "#PWR2" H 725 3025 50  0001 C CNN
+F 0 "#PWR012" H 725 3025 50  0001 C CNN
 F 1 "GND" H 725 3125 50  0000 C CNN
 F 2 "" H 725 3275 50  0000 C CNN
@@
 $EndComp
 $Comp
-L +3.3V #PWR3
+L +3.3V #PWR013
 U 1 1 5A62AFDE
 P 1650 2425
-F 0 "#PWR3" H 1650 2275 50  0001 C CNN
+F 0 "#PWR013" H 1650 2275 50  0001 C CNN
 F 1 "+3.3V" H 1650 2565 50  0000 C CNN
 F 2 "" H 1650 2425 50  0001 C CNN
@@
 $EndSheet
 $Comp
-L +3.3V #PWR22
+L +3.3V #PWR014
 U 1 1 5A6EE2A3
 P 9250 3575
-F 0 "#PWR22" H 9250 3425 50  0001 C CNN
+F 0 "#PWR014" H 9250 3425 50  0001 C CNN
 F 1 "+3.3V" H 9250 3715 50  0000 C CNN
 F 2 "" H 9250 3575 50  0001 C CNN
@@
 $EndComp
 $Comp
-L GND #PWR21
+L GND #PWR015
 U 1 1 5A6F9F51
 P 9250 1825
-F 0 "#PWR21" H 9250 1575 50  0001 C CNN
+F 0 "#PWR015" H 9250 1575 50  0001 C CNN
 F 1 "GND" H 9250 1675 50  0000 C CNN
 F 2 "" H 9250 1825 50  0001 C CNN
@@
 NoConn ~ 8325 1175
 $Comp
-L +3.3V #PWR12
+L +3.3V #PWR016
 U 1 1 5A83C4F3
 P 4550 1300
-F 0 "#PWR12" H 4550 1150 50  0001 C CNN
+F 0 "#PWR016" H 4550 1150 50  0001 C CNN
 F 1 "+3.3V" H 4550 1440 50  0000 C CNN
 F 2 "" H 4550 1300 50  0001 C CNN
@@
 Connection ~ 6575 2050
 $Comp
-L +5V #PWR13
+L +5V #PWR017
 U 1 1 5A9E0ED0
 P 6300 2050
-F 0 "#PWR13" H 6300 1900 50  0001 C CNN
+F 0 "#PWR017" H 6300 1900 50  0001 C CNN
 F 1 "+5V" H 6300 2190 50  0000 C CNN
 F 2 "" H 6300 2050 50  0001 C CNN
@@
 Connection ~ 6775 2850
 $Comp
-L GND #PWR14
+L GND #PWR018
 U 1 1 5A9E143E
 P 7100 2850
-F 0 "#PWR14" H 7100 2600 50  0001 C CNN
+F 0 "#PWR018" H 7100 2600 50  0001 C CNN
 F 1 "GND" H 7100 2700 50  0000 C CNN
 F 2 "" H 7100 2850 50  0001 C CNN
@@
 F 0 "U4" H 7875 2825 60  0000 C CNN
 F 1 "IS31FL3733" H 7875 5825 60  0000 C CNN
-F 2 "" H 7875 4775 60  0001 C CNN
+F 2 "Housings_DFN_QFN:QFN-48-1EP_6x6mm_Pitch0.4mm" H 7875 4775 60  0001 C CNN
 F 3 "" H 7875 4775 60  0001 C CNN
 	1    7875 4475
@@
 Connection ~ 8475 3675
 $Comp
-L +5V #PWR15
+L +5V #PWR019
 U 1 1 5A9E3817
 P 8475 3575
-F 0 "#PWR15" H 8475 3425 50  0001 C CNN
+F 0 "#PWR019" H 8475 3425 50  0001 C CNN
 F 1 "+5V" H 8475 3715 50  0000 C CNN
 F 2 "" H 8475 3575 50  0001 C CNN
@@
 	8375 5675 8925 5675
 $Comp
-L GND #PWR17
+L GND #PWR020
 U 1 1 5A9E3BA4
 P 8525 5875
-F 0 "#PWR17" H 8525 5625 50  0001 C CNN
+F 0 "#PWR020" H 8525 5625 50  0001 C CNN
 F 1 "GND" H 8525 5725 50  0000 C CNN
 F 2 "" H 8525 5875 50  0001 C CNN
@@
 Connection ~ 8525 5675
 $Comp
-L +3.3V #PWR18
+L +3.3V #PWR021
 U 1 1 5A9E3CE2
 P 8925 5600
-F 0 "#PWR18" H 8925 5450 50  0001 C CNN
+F 0 "#PWR021" H 8925 5450 50  0001 C CNN
 F 1 "+3.3V" H 8925 5740 50  0000 C CNN
 F 2 "" H 8925 5600 50  0001 C CNN
@@
 Connection ~ 8525 5375
 $Comp
-L GND #PWR16
+L GND #PWR022
 U 1 1 5A9E4271
 P 8525 5475
-F 0 "#PWR16" H 8525 5225 50  0001 C CNN
+F 0 "#PWR022" H 8525 5225 50  0001 C CNN
 F 1 "GND" H 8525 5325 50  0000 C CNN
 F 2 "" H 8525 5475 50  0001 C CNN
@@
 	8675 4475 8375 4475
 $Comp
-L GND #PWR19
+L GND #PWR023
 U 1 1 5A9E51CA
 P 9000 4475
-F 0 "#PWR19" H 9000 4225 50  0001 C CNN
+F 0 "#PWR023" H 9000 4225 50  0001 C CNN
 F 1 "GND" H 9000 4325 50  0000 C CNN
 F 2 "" H 9000 4475 50  0001 C CNN

Commit message: Revert LED structure
Parts:
- C1, C10, C11, C12, C13, C14, C2, C3, C4, C5, C6, C7, C8, C9: footprint Capacitors_SMD:C_0805 -> Capacitors_SMD:C_0603
- R1, R2, R3, R4, R6, R7, R8: footprint Resistors_SMD:R_0805 -> Resistors_SMD:R_0603
Changed lines of the file:
@@
 F 0 "C1" H 4310 1470 50  0000 L CNN
 F 1 "1u" H 4310 1320 50  0000 L CNN
-F 2 "Capacitors_SMD:C_0805" H 4300 1400 50  0001 C CNN
+F 2 "Capacitors_SMD:C_0603" H 4300 1400 50  0001 C CNN
 F 3 "" H 4300 1400 50  0001 C CNN
 	1    4300 1400
@@
 F 0 "C2" H 735 3245 50  0000 L CNN
 F 1 "0.1u" H 735 3095 50  0000 L CNN
-F 2 "Capacitors_SMD:C_0805" H 725 3175 50  0001 C CNN
+F 2 "Capacitors_SMD:C_0603" H 725 3175 50  0001 C CNN
 F 3 "" H 725 3175 50  0000 C CNN
 	1    725  3175
@@
 F 0 "C4" H 1135 3245 50  0000 L CNN
 F 1 "0.1u" H 1135 3095 50  0000 L CNN
-F 2 "Capacitors_SMD:C_0805" H 1125 3175 50  0001 C CNN
+F 2 "Capacitors_SMD:C_0603" H 1125 3175 50  0001 C CNN
 F 3 "" H 1125 3175 50  0000 C CNN
 	1    1125 3175
@@
 F 0 "C5" H 1335 3245 50  0000 L CNN
 F 1 "0.1u" H 1335 3095 50  0000 L CNN
-F 2 "Capacitors_SMD:C_0805" H 1325 3175 50  0001 C CNN
+F 2 "Capacitors_SMD:C_0603" H 1325 3175 50  0001 C CNN
 F 3 "" H 1325 3175 50  0000 C CNN
 	1    1325 3175
@@
 F 0 "C3" H 935 3245 50  0000 L CNN
 F 1 "0.1u" H 935 3095 50  0000 L CNN
-F 2 "Capacitors_SMD:C_0805" H 925 3175 50  0001 C CNN
+F 2 "Capacitors_SMD:C_0603" H 925 3175 50  0001 C CNN
 F 3 "" H 925 3175 50  0000 C CNN
 	1    925  3175
@@
 F 0 "C6" H 1560 3245 50  0000 L CNN
 F 1 "10u" H 1560 3095 50  0000 L CNN
-F 2 "Capacitors_SMD:C_0805" H 1550 3175 50  0001 C CNN
+F 2 "Capacitors_SMD:C_0603" H 1550 3175 50  0001 C CNN
 F 3 "" H 1550 3175 50  0000 C CNN
 	1    1550 3175
@@
 F 0 "R1" H 2580 2420 50  0000 L CNN
 F 1 "10k" H 2580 2360 50  0000 L CNN
-F 2 "Resistors_SMD:R_0805" H 2550 2400 50  0001 C CNN
+F 2 "Resistors_SMD:R_0603" H 2550 2400 50  0001 C CNN
 F 3 "" H 2550 2400 50  0000 C CNN
 	1    2550 2400
@@
 F 0 "C8" H 6585 2220 50  0000 L CNN
 F 1 "0.1u" H 6585 2070 50  0000 L CNN
-F 2 "Capacitors_SMD:C_0805" H 6575 2150 50  0001 C CNN
+F 2 "Capacitors_SMD:C_0603" H 6575 2150 50  0001 C CNN
 F 3 "" H 6575 2150 50  0001 C CNN
 	1    6575 2150
@@
 F 0 "C7" H 7110 2220 50  0000 L CNN
 F 1 "10u" H 7110 2070 50  0000 L CNN
-F 2 "Capacitors_SMD:C_0805" H 7100 2150 50  0001 C CNN
+F 2 "Capacitors_SMD:C_0603" H 7100 2150 50  0001 C CNN
 F 3 "" H 7100 2150 50  0001 C CNN
 	1    7100 2150
@@
 F 0 "R3" H 9280 3795 50  0000 L CNN
 F 1 "1k" H 9280 3735 50  0000 L CNN
-F 2 "Resistors_SMD:R_0805" H 9250 3775 50  0001 C CNN
+F 2 "Resistors_SMD:R_0603" H 9250 3775 50  0001 C CNN
 F 3 "" H 9250 3775 50  0001 C CNN
 	1    9250 3775
@@
 F 0 "R4" H 9455 3795 50  0000 L CNN
 F 1 "1k" H 9455 3735 50  0000 L CNN
-F 2 "Resistors_SMD:R_0805" H 9425 3775 50  0001 C CNN
+F 2 "Resistors_SMD:R_0603" H 9425 3775 50  0001 C CNN
 F 3 "" H 9425 3775 50  0001 C CNN
 	1    9425 3775
@@
 F 0 "R6" V 8850 2250 50  0000 L CNN
 F 1 "5.1k" V 8850 2375 50  0000 L CNN
-F 2 "Resistors_SMD:R_0805" H 8925 2375 50  0001 C CNN
+F 2 "Resistors_SMD:R_0603" H 8925 2375 50  0001 C CNN
 F 3 "" H 8925 2375 50  0001 C CNN
 	1    8925 2375
@@
 F 0 "R7" V 8850 2350 50  0000 L CNN
 F 1 "5.1k" V 8850 2475 50  0000 L CNN
-F 2 "Resistors_SMD:R_0805" H 8925 2475 50  0001 C CNN
+F 2 "Resistors_SMD:R_0603" H 8925 2475 50  0001 C CNN
 F 3 "" H 8925 2475 50  0001 C CNN
 	1    8925 2475
@@
 F 0 "C11" H 6785 2220 50  0000 L CNN
 F 1 "0.47u" H 6785 2070 50  0000 L CNN
-F 2 "Capacitors_SMD:C_0805" H 6775 2150 50  0001 C CNN
+F 2 "Capacitors_SMD:C_0603" H 6775 2150 50  0001 C CNN
 F 3 "" H 6775 2150 50  0001 C CNN
 	1    6775 2150
@@
 F 0 "C9" H 6585 2520 50  0000 L CNN
 F 1 "0.1u" H 6585 2370 50  0000 L CNN
-F 2 "Capacitors_SMD:C_0805" H 6575 2450 50  0001 C CNN
+F 2 "Capacitors_SMD:C_0603" H 6575 2450 50  0001 C CNN
 F 3 "" H 6575 2450 50  0001 C CNN
 	1    6575 2450
@@
 F 0 "C12" H 6785 2520 50  0000 L CNN
 F 1 "0.47u" H 6785 2370 50  0000 L CNN
-F 2 "Capacitors_SMD:C_0805" H 6775 2450 50  0001 C CNN
+F 2 "Capacitors_SMD:C_0603" H 6775 2450 50  0001 C CNN
 F 3 "" H 6775 2450 50  0001 C CNN
 	1    6775 2450
@@
 F 0 "C10" H 6585 2820 50  0000 L CNN
 F 1 "0.1u" H 6585 2670 50  0000 L CNN
-F 2 "Capacitors_SMD:C_0805" H 6575 2750 50  0001 C CNN
+F 2 "Capacitors_SMD:C_0603" H 6575 2750 50  0001 C CNN
 F 3 "" H 6575 2750 50  0001 C CNN
 	1    6575 2750
@@
 F 0 "C13" H 6785 2820 50  0000 L CNN
 F 1 "0.47u" H 6785 2670 50  0000 L CNN
-F 2 "Capacitors_SMD:C_0805" H 6775 2750 50  0001 C CNN
+F 2 "Capacitors_SMD:C_0603" H 6775 2750 50  0001 C CNN
 F 3 "" H 6775 2750 50  0001 C CNN
 	1    6775 2750
@@
 F 0 "C14" H 8535 5845 50  0000 L CNN
 F 1 "0.47u" H 8535 5695 50  0000 L CNN
-F 2 "Capacitors_SMD:C_0805" H 8525 5775 50  0001 C CNN
+F 2 "Capacitors_SMD:C_0603" H 8525 5775 50  0001 C CNN
 F 3 "" H 8525 5775 50  0001 C CNN
 	1    8525 5775
@@
 F 0 "R8" H 9230 4895 50  0000 L CNN
 F 1 "20k" H 9230 4835 50  0000 L CNN
-F 2 "Resistors_SMD:R_0805" H 9200 4875 50  0001 C CNN
+F 2 "Resistors_SMD:R_0603" H 9200 4875 50  0001 C CNN
 F 3 "" H 9200 4875 50  0001 C CNN
 	1    9200 4875
@@
 F 0 "R2" H 8805 4495 50  0000 L CNN
 F 1 "100k" H 8805 4435 50  0000 L CNN
-F 2 "Resistors_SMD:R_0805" H 8775 4475 50  0001 C CNN
+F 2 "Resistors_SMD:R_0603" H 8775 4475 50  0001 C CNN
 F 3 "" H 8775 4475 50  0001 C CNN
 	1    8775 4475

Commit message: Begin routing
Connections:
- net LED-CS1: now reaches U4.16 (CS1)
- net LED-CS2: now reaches U4.17 (CS2)
- net LED-CS3: now reaches U4.18 (CS3)
- net LED-CS4: now reaches U4.19 (CS4)
- net LED-SW1: now reaches U4.2 (SW1)
- net LED-CS5: now reaches U4.21 (CS5)
- net LED-CS6: now reaches U4.22 (CS6)
- net LED-CS7: now reaches U4.23 (CS7)
- net LED-CS8: now reaches U4.24 (CS8)
- net LED-CS9: now reaches U4.25 (CS9)
- net LED-CS10: now reaches U4.26 (CS10)
- net LED-CS11: now reaches U4.27 (CS11)
- net LED-CS12: now reaches U4.28 (CS12)
- net LED-SW2: now reaches U4.3 (SW2)
- net LED-CS13: now reaches U4.30 (CS13)
- net LED-CS14: now reaches U4.31 (CS14)
- net LED-CS15: now reaches U4.32 (CS15)
- net LED-SW3: now reaches U4.4 (SW3)
- net LED-SW4: now reaches U4.6 (SW4)
- net LED-SW5: now reaches U4.7 (SW5)
Changed lines of the file:
@@
 NoConn ~ 8375 3275
 NoConn ~ 8375 3375
+Text GLabel 7375 4475 0    60   Input ~ 0
+LED-CS1
+Text GLabel 7375 4575 0    60   Input ~ 0
+LED-CS2
+Text GLabel 7375 4675 0    60   Input ~ 0
+LED-CS3
+Text GLabel 7375 4775 0    60   Input ~ 0
+LED-CS4
+Text GLabel 7375 4875 0    60   Input ~ 0
+LED-CS5
+Text GLabel 7375 4975 0    60   Input ~ 0
+LED-CS6
+Text GLabel 7375 5075 0    60   Input ~ 0
+LED-CS7
+Text GLabel 7375 5175 0    60   Input ~ 0
+LED-CS8
+Text GLabel 7375 5275 0    60   Input ~ 0
+LED-CS9
+Text GLabel 7375 5375 0    60   Input ~ 0
+LED-CS10
+Text GLabel 7375 5475 0    60   Input ~ 0
+LED-CS11
+Text GLabel 7375 5575 0    60   Input ~ 0
+LED-CS12
+Text GLabel 7375 5675 0    60   Input ~ 0
+LED-CS13
+Text GLabel 7375 5775 0    60   Input ~ 0
+LED-CS14
+Text GLabel 7375 5875 0    60   Input ~ 0
+LED-CS15
+Text GLabel 7375 3275 0    60   Input ~ 0
+LED-SW1
+Text GLabel 7375 3375 0    60   Input ~ 0
+LED-SW2
+Text GLabel 7375 3475 0    60   Input ~ 0
+LED-SW3
+Text GLabel 7375 3575 0    60   Input ~ 0
+LED-SW4
+Text GLabel 7375 3675 0    60   Input ~ 0
+LED-SW5
 $EndSCHEMATC

Commit message: Tune up routing
Connections:
- net +3V3: now also U4.46 (SDB)
Other:
- note added: "SDA and SCL are marked as I2C+- for the sake of using KiCad's differential router"
Changed lines of the file:
@@
 Text GLabel 7375 3675 0    60   Input ~ 0
 LED-SW5
+Text Notes 2675 5400 0    60   ~ 0
+SDA and SCL are marked as I2C+- for the sake of using KiCad's differential router
+$Comp
+L +3.3V #PWR?
+U 1 1 5AA88312
+P 8575 4375
+F 0 "#PWR?" H 8575 4225 50  0001 C CNN
+F 1 "+3.3V" H 8575 4515 50  0000 C CNN
+F 2 "" H 8575 4375 50  0001 C CNN
+F 3 "" H 8575 4375 50  0001 C CNN
+	1    8575 4375
+	1    0    0    -1
+$EndComp
+Wire Wire Line
+	8575 4375 8375 4375
 $EndSCHEMATC

Commit message: Tune routing
Connections:
- no-connect marks 4 -> 6
Changed lines of the file:
@@
 Wire Wire Line
 	8575 4375 8375 4375
+NoConn ~ 1100 2525
+NoConn ~ 1600 2525
 $EndSCHEMATC
