File: Voyager65.kicad_pcb (KiCad board)
At the start: 2 copper layers, 285 x 95.1 mm, 197 parts, among them P1 TC2030-IDC, SW1 SW_PUSH, U1 ATXMEGA32A4U-AU, U2 MCP1700T-3002E/TT, U3 PRTR5V0U2X, U4 IS31FL3733, U5 74LVC1G34

Commit message: Replace MCU, route bus
Parts:
- removed LM1, LM4, RM1: MX-1.5U, MX_Alps_Hybrid:MX-1.5U
- removed LM2, RM4, RM7, RM9, RS1, RS5, RS6: MX-1U, MX_Alps_Hybrid:MX-1U
- removed LM3: MX-1.25U, MX_Alps_Hybrid:MX-1.25U-FLIPPED
- removed LM5, RM8: MX-1.5U, MX_Alps_Hybrid:MX-1.5U-FLIPPED
- removed the REF** at (190.5, 95.2)
- removed RM2, RM6: MX-1U, MX_Alps_Hybrid:MX-1U-FLIPPED
- removed RM3, RM5: MX-1.25U, MX_Alps_Hybrid:MX-1.25U
- removed RS2: MX-2.75U, MX_Alps_Hybrid:MX-2.75U-FLIPPED
- removed RS3, RS4: MX-1.75U, MX_Alps_Hybrid:MX-1.75U
- added D45: D_Small, Diodes_SMD:D_SOD-123, B.Cu at (335.0, 76.2)
- added D65: D_Small, Diodes_SMD:D_SOD-123, B.Cu at (121.4, 133.3)
- added D66: D_Small, Diodes_SMD:D_SOD-123, B.Cu at (157.2, 133.3)
- added D67: D_Small, Diodes_SMD:D_SOD-123, B.Cu at (197.6, 133.3)
- added D68: D_Small, Diodes_SMD:D_SOD-123, B.Cu at (233.4, 133.3)
- added D69: D_Small, Diodes_SMD:D_SOD-123, B.Cu at (239.7, 133.3)
- added D70: D_Small, Diodes_SMD:D_SOD-123, B.Cu at (296.9, 133.3)
- added D71: D_Small, Diodes_SMD:D_SOD-123, B.Cu at (292.9, 133.3)
- added K_/1: MX-1U, MX_Alps_Hybrid:MX-1U, F.Cu at (271.5, 114.3)
- added K_DOWN1: MX-1U, MX_Alps_Hybrid:MX-1U, F.Cu at (323.9, 133.3)
- added K_EX1: MX-1U, MX_Alps_Hybrid:MX-1U, F.Cu at (342.9, 57.1)
- added K_EX2: MX-1U, MX_Alps_Hybrid:MX-1U, F.Cu at (342.9, 76.2)
- added K_EX3: MX-1U, MX_Alps_Hybrid:MX-1U, F.Cu at (342.9, 95.2)
- added K_EX4: MX-1U, MX_Alps_Hybrid:MX-1U, F.Cu at (342.9, 114.3)
- added K_LEFT1: MX-1U, MX_Alps_Hybrid:MX-1U, F.Cu at (304.8, 133.3)
- added K_LM1: MX-1.5U, MX_Alps_Hybrid:MX-1.5U, F.Cu at (61.9, 133.3)
- added K_LM2: MX-1.25U, MX_Alps_Hybrid:MX-1.25U-FLIPPED, F.Cu at (59.5, 133.3)
- added K_LM3: MX-1.5U, MX_Alps_Hybrid:MX-1.5U-FLIPPED, F.Cu at (90.5, 133.3)
- added K_LM4: MX-1.25U, MX_Alps_Hybrid:MX-1.25U, F.Cu at (83.3, 133.3)
- added K_LM5: MX-1.25U, MX_Alps_Hybrid:MX-1.25U, F.Cu at (88.1, 133.3)
- added K_LM6: MX-1.25U, MX_Alps_Hybrid:MX-1.25U, F.Cu at (107.2, 133.3)
- added K_LM7: MX-1.5U, MX_Alps_Hybrid:MX-1.5U, F.Cu at (114.3, 133.3)
- added K_RIGHT1: MX-1U, MX_Alps_Hybrid:MX-1U, F.Cu at (342.9, 133.3)
- added K_RM1: MX-1U, MX_Alps_Hybrid:MX-1U, F.Cu at (247.7, 133.3)
- added K_RM2: MX-1.5U, MX_Alps_Hybrid:MX-1.5U, F.Cu at (252.4, 133.3)
- added K_RM3: MX-1.25U, MX_Alps_Hybrid:MX-1.25U, F.Cu at (264.3, 133.3)
- added K_RM4: MX-1U, MX_Alps_Hybrid:MX-1U, F.Cu at (266.7, 133.3)
- added K_RM5: MX-1.5U, MX_Alps_Hybrid:MX-1.5U, F.Cu at (281.0, 133.3)
- added K_RM6: MX-1U, MX_Alps_Hybrid:MX-1U, F.Cu at (285.8, 133.3)
- added K_SHIFT2: MX-1.75U, MX_Alps_Hybrid:MX-1.75U, F.Cu at (297.7, 114.3)
- added K_UP1: MX-1U, MX_Alps_Hybrid:MX-1U, F.Cu at (323.9, 114.3)
- added SP2: MX-7U, MX_Alps_Hybrid:MX-7U-ReversedStabilizers, F.Cu at (171.4, 133.3)
- added SP3: MX-6.25U, MX_Alps_Hybrid:MX-6.25U-ReversedStabilizers, F.Cu at (178.6, 133.3)
- added SP4: MX-1.25U, MX_Alps_Hybrid:MX-1.25U, F.Cu at (173.8, 133.3)
- added SP5: MX-2.75U, MX_Alps_Hybrid:MX-2.75U-ReversedStabilizers, F.Cu at (211.9, 133.3)
- added SP6: MX-6.5U, MX_Alps_Hybrid:MX-6.5U-ReversedStabilizers, F.Cu at (190.5, 133.3)
- added SP7: MX-2.25U, MX_Alps_Hybrid:MX-2.25U-ReversedStabilizers, F.Cu at (150.0, 133.3)
- added SP8: MX-1.5U, MX_Alps_Hybrid:MX-1.5U, F.Cu at (185.7, 133.3)
- added SP9: MX-2.75U, MX_Alps_Hybrid:MX-2.75U-ReversedStabilizers, F.Cu at (226.2, 133.3)
- SP1: value MX-7U -> MX-2.25U; footprint MX_Alps_Hybrid:MX-7U-ReversedStabilizers -> MX_Alps_Hybrid:MX-2.25U-ReversedStabilizers
- U1: footprint Housings_QFP:TQFP-44_10x10mm_Pitch0.8mm -> Housings_DFN_QFN:QFN-44-1EP_7x7mm_Pitch0.5mm
- moved LED9 285.9 mm to (26.0, 103.5), turned to 0 degrees
- moved CRGB9 285.2 mm to (32.4, 103.2), turned to 0 degrees
- moved LED7 284.3 mm to (26.0, 103.5), turned to 0 degrees
- moved CRGB7 272.2 mm to (32.4, 103.2), turned to 0 degrees
- moved D63 242.9 mm to (69.1, 133.3)
- moved D60 242.9 mm to (311.9, 133.3)
- moved LED11 238.8 mm to (26.0, 103.5), turned to 0 degrees
- moved CRGB11 238.0 mm to (32.4, 103.2), turned to 0 degrees
- moved LED5 236.8 mm to (26.0, 103.5), turned to 0 degrees
- moved D61 235.7 mm to (331.0, 133.3)
- moved CRGB5 224.7 mm to (32.4, 103.2), turned to 0 degrees
- moved D64 214.3 mm to (97.6, 133.3), turned to 90 degrees
- moved D62 213.5 mm to (335.0, 133.3)
- moved LED2 191.8 mm to (26.0, 103.5), turned to 0 degrees
- moved CRGB2 191.1 mm to (32.4, 103.2), turned to 0 degrees
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Connections:
- D42 pad 1: ROW4 -> ROW0
- D55 pad 1: ROW4 -> ROW2
- D56 pad 1: ROW4 -> ROW3
- SP1 pad 1: COL6 -> Net-(SP1-Pad1)
- SP1 pad 2: Net-(D55-Pad2) -> Net-(D66-Pad2)
- SP1 pad 3: LED-CS7 -> Net-(SP1-Pad3)
- SP1 pad 4: LED-SW1 -> Net-(SP1-Pad4)
- U1 pad 37: Net-(U1-Pad37) -> COL15
- U4 pad 33: Net-(U4-Pad33) -> LED-CS16
Routing:
- net GND: track 2243.7 -> 414.3 mm, vias 76 -> 10
- net +5V: track 873.0 -> 48.4 mm, vias 14 -> 3
- net COL15: track 0.00 -> 354.9 mm
- net LED-SW1: track 340.9 -> 21.0 mm, vias 3 -> 1
- net ROW4: track 271.0 -> 3.67 mm, vias 4 -> 0
- net I2C+: track 186.2 -> 1.80 mm, vias 4 -> 1
- net I2C-: track 184.4 -> 2.31 mm, vias 4 -> 1
- net +3V3: track 255.6 -> 85.2 mm, vias 4 -> 5
- net LED-CS16: track 0.00 -> 135.3 mm
- net PDI_CLK: track 136.9 -> 4.43 mm, vias 2 -> 0
- net D+: track 147.7 -> 39.0 mm
- net D-: track 149.4 -> 41.3 mm
- net COL0: track 191.9 -> 102.7 mm
- net ROW0: track 375.2 -> 290.5 mm, vias 6 -> 4
- net ROW3: track 273.0 -> 193.1 mm, vias 6 -> 0
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- removed copper zone on B.Cu, net GND
Other:
- board size 285 x 95.1 mm -> 304.8 x 95.2 mm
- net class Default: clearance 0.1524 -> 0.254
- net class Power: clearance 0.1524 -> 0.254
- rule trace_clearance: 0.1524 -> 0.254
- board text added: "65"
- board text removed: "Revision 2"

Commit message: A few more traces before I sleep
Routing:
- net LED-CS14: track 50.8 -> 98.8 mm, vias 0 -> 1
- net LED-CS15: track 102.5 -> 124.0 mm
- net COL13: track 277.5 -> 278.3 mm
- net COL14: track 346.0 -> 346.7 mm
Changed lines of the file:
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@@
     (thickness 1.6)
     (drawings 48)
-    (tracks 1884)
+    (tracks 1902)
     (zones 0)
     (modules 215)
@@
   (segment (start 66.675 62.561) (end 67.421 63.307) (width 0.254) (layer B.Cu) (net 28) (status 20))
   (segment (start 65.9876 54.195) (end 65.9876 55.7006) (width 0.254) (layer B.Cu) (net 28) (status 10))
+  (segment (start 320.04 111.76) (end 320.802 112.522) (width 0.254) (layer F.Cu) (net 32))
+  (segment (start 320.802 112.522) (end 320.802 130.048) (width 0.254) (layer F.Cu) (net 32))
+  (segment (start 320.802 130.048) (end 320.04 130.81) (width 0.254) (layer F.Cu) (net 32))
   (segment (start 317.246 109.093) (end 308.13375 99.98075) (width 0.254) (layer F.Cu) (net 32))
   (segment (start 321.35 110.276) (end 320.167 109.093) (width 0.254) (layer F.Cu) (net 32))
   (segment (start 320.167 109.093) (end 317.246 109.093) (width 0.254) (layer F.Cu) (net 32))
   (segment (start 321.35 110.3) (end 321.35 110.276) (width 0.254) (layer F.Cu) (net 32))
-  (segment (start 320.04 111.76) (end 320.04 130.81) (width 0.254) (layer F.Cu) (net 32))
   (segment (start 320.04 111.76) (end 319.913 111.76) (width 0.254) (layer F.Cu) (net 32))
   (segment (start 308.13375 99.98075) (end 308.13375 92.71) (width 0.254) (layer F.Cu) (net 32))
@@
   (segment (start 320.675 56.596786) (end 320.675 68.1125) (width 0.254) (layer F.Cu) (net 32))
   (segment (start 320.675 68.1125) (end 316.5875 72.2) (width 0.254) (layer F.Cu) (net 32) (status 20))
+  (segment (start 303.276 107.823) (end 304.038 108.585) (width 0.254) (layer F.Cu) (net 33))
+  (segment (start 304.038 108.585) (end 304.038 129.032) (width 0.254) (layer F.Cu) (net 33))
+  (segment (start 304.038 129.032) (end 303.72 129.35) (width 0.254) (layer F.Cu) (net 33))
+  (segment (start 303.72 129.35) (end 302.3 129.35) (width 0.254) (layer F.Cu) (net 33))
   (segment (start 80.616 90.1326) (end 81.7506 90.1326) (width 0.254) (layer B.Cu) (net 33))
   (segment (start 81.7506 90.1326) (end 83.058 91.44) (width 0.254) (layer B.Cu) (net 33))
@@
   (segment (start 276.987 107.569) (end 303.022 107.569) (width 0.254) (layer B.Cu) (net 33))
   (segment (start 303.022 107.569) (end 303.276 107.823) (width 0.254) (layer B.Cu) (net 33))
-  (segment (start 304.038 108.585) (end 304.038 127.612) (width 0.254) (layer F.Cu) (net 33))
-  (segment (start 304.038 127.612) (end 302.3 129.35) (width 0.254) (layer F.Cu) (net 33))
-  (segment (start 303.276 107.823) (end 304.038 108.585) (width 0.254) (layer F.Cu) (net 33))
   (via (at 303.276 107.823) (size 0.6) (drill 0.4) (layers F.Cu B.Cu) (net 33))
   (segment (start 291.465 73.66) (end 291.465 73.914) (width 0.254) (layer F.Cu) (net 33) (status 30))
@@
   (segment (start 261.112 90.551) (end 255.905 85.344) (width 0.254) (layer F.Cu) (net 140))
   (segment (start 255.905 85.344) (end 255.905 81.28) (width 0.254) (layer F.Cu) (net 140) (status 20))
+  (segment (start 322.58 119.38) (end 321.31 120.65) (width 0.254) (layer F.Cu) (net 141))
+  (segment (start 321.31 120.65) (end 321.31 126.873) (width 0.254) (layer F.Cu) (net 141))
+  (segment (start 321.31 126.873) (end 323.088 128.651) (width 0.254) (layer F.Cu) (net 141))
+  (segment (start 323.088 128.651) (end 323.088 130.175) (width 0.254) (layer F.Cu) (net 141))
+  (segment (start 323.088 130.175) (end 321.31 131.953) (width 0.254) (layer F.Cu) (net 141))
+  (segment (start 321.31 131.953) (end 321.31 137.16) (width 0.254) (layer F.Cu) (net 141))
+  (segment (start 321.31 137.16) (end 322.58 138.43) (width 0.254) (layer F.Cu) (net 141))
   (segment (start 294.198 96.104) (end 295.748 96.104) (width 0.2032) (layer B.Cu) (net 141))
   (segment (start 297.053 97.409) (end 308.737 97.409) (width 0.254) (layer B.Cu) (net 141))
@@
   (segment (start 66.548 112.776) (end 68.199 111.125) (width 0.254) (layer F.Cu) (net 142))
   (segment (start 60.80125 100.33) (end 63.02375 100.33) (width 0.254) (layer B.Cu) (net 142) (status 30))
+  (segment (start 303.53 138.43) (end 302.26 137.16) (width 0.254) (layer F.Cu) (net 143))
+  (segment (start 302.26 137.16) (end 302.26 131.953) (width 0.254) (layer F.Cu) (net 143))
+  (segment (start 302.26 131.953) (end 304.546 129.667) (width 0.254) (layer F.Cu) (net 143))
+  (segment (start 304.546 129.667) (end 304.546 96.901) (width 0.254) (layer F.Cu) (net 143))
+  (segment (start 304.546 96.901) (end 301.498 93.853) (width 0.254) (layer F.Cu) (net 143))
+  (segment (start 301.498 93.853) (end 301.498 93.599) (width 0.254) (layer F.Cu) (net 143))
+  (segment (start 301.244 93.853) (end 301.498 93.599) (width 0.254) (layer B.Cu) (net 143))
+  (via (at 301.498 93.599) (size 0.6) (drill 0.4) (layers F.Cu B.Cu) (net 143))
   (segment (start 297.307 96.901) (end 300.863 96.901) (width 0.254) (layer B.Cu) (net 143))
   (segment (start 300.863 96.901) (end 301.244 96.52) (width 0.254) (layer B.Cu) (net 143))
@@
     (connect_pads (clearance 0.3556))
     (min_thickness 0.254)
-    (fill (arc_segments 16) (thermal_gap 0.508) (thermal_bridge_width 0.508))
+    (fill yes (arc_segments 16) (thermal_gap 0.508) (thermal_bridge_width 0.508))
     (polygon
       (pts

Commit message: Sleep
Parts:
- moved LED2 104.5 mm to (123.8, 66.7), turned to 90 degrees
- moved LED1 68.1 mm to (83.3, 66.7), turned to 90 degrees
- moved R5 34.9 mm to (43.8, 73.8)
- moved U5 34.9 mm to (43.8, 77.1)
Routing:
- net LED-CS1: track 312.1 -> 310.3 mm

Commit message: Temporary progress save
Parts:
- K_LM4: footprint MX_Alps_Hybrid:MX-1.25U -> MX_Alps_Hybrid:MX-1.25U-FLIPPED
- K_RM2: footprint MX_Alps_Hybrid:MX-1.5U -> MX_Alps_Hybrid:MX-1.5U-FLIPPED
- K_RM4, K_RM6: footprint MX_Alps_Hybrid:MX-1U -> MX_Alps_Hybrid:MX-1U-FLIPPED
- moved CRGB2 300.9 mm to (332.6, 123.8), turned to 270 degrees
- moved LED11 296.1 mm to (319.9, 66.7), turned to 90 degrees
- moved CRGB11 284.3 mm to (314.3, 66.7), turned to 270 degrees
- moved LED9 252.9 mm to (276.2, 66.7), turned to 90 degrees
- moved CRGB9 252.1 mm to (281.8, 66.7), turned to 270 degrees
- moved LED4 246.3 mm to (271.5, 123.8), turned to 90 degrees
- moved CRGB4 245.5 mm to (277.0, 123.8), turned to 270 degrees
- moved LED2 211.1 mm to (327.0, 123.8)
- moved LED7 202.8 mm to (225.4, 66.7), turned to 90 degrees
- moved CRGB7 201.9 mm to (231.0, 66.7), turned to 270 degrees
- moved CRGB6 186.2 mm to (217.5, 123.8), turned to 270 degrees
- moved LED6 183.1 mm to (208.0, 123.8), turned to 90 degrees
- moved LED5 153.1 mm to (174.6, 66.7), turned to 90 degrees
- moved CRGB5 152.2 mm to (180.2, 66.7), turned to 270 degrees
- moved LED8 143.7 mm to (168.3, 123.8), turned to 90 degrees
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Connections:
- D69 pad 1: Net-(D69-Pad1) -> ROW4
- D70 pad 1: Net-(D70-Pad1) -> ROW4
- D71 pad 1: Net-(D71-Pad1) -> ROW4
- K_LM5 pad 2: Net-(K_LM5-Pad2) -> Net-(D64-Pad2)
- K_RM1 pad 1: Net-(K_RM1-Pad1) -> COL10
- K_RM2 pad 1: Net-(K_RM2-Pad1) -> Net-(D69-Pad2)
- K_RM2 pad 2: Net-(K_RM2-Pad2) -> COL10
- K_RM3 pad 1: Net-(K_RM3-Pad1) -> COL11
- K_RM4 pad 1: Net-(K_RM4-Pad1) -> COL11
- K_RM4 pad 2: Net-(K_RM4-Pad2) -> Net-(D70-Pad2)
- K_RM5 pad 1: Net-(K_RM5-Pad1) -> COL12
- K_RM6 pad 1: Net-(K_RM6-Pad1) -> Net-(D71-Pad2)
- K_RM6 pad 2: Net-(K_RM6-Pad2) -> COL12
Routing:
- net +5V: track 48.4 -> 751.8 mm, vias 3 -> 24
- net GND: track 414.3 -> 998.7 mm, vias 10 -> 17
- net ROW4: track 3.67 -> 79.9 mm
- net Net-(LED4-Pad2): track 0.00 -> 70.7 mm
- net Net-(LED2-Pad2): track 0.00 -> 62.8 mm
- net Net-(LED10-Pad2): track 0.00 -> 57.2 mm
- net Net-(LED10-Pad4): track 0.00 -> 53.3 mm
- net COL12: track 267.1 -> 315.5 mm, vias 0 -> 1
- net Net-(LED7-Pad2): track 0.00 -> 47.4 mm
- net Net-(LED5-Pad2): track 0.00 -> 47.4 mm
- net Net-(LED3-Pad2): track 0.00 -> 47.4 mm
- net Net-(LED6-Pad2): track 0.00 -> 46.9 mm
- net Net-(LED11-Pad4): track 0.00 -> 41.9 mm
- net Net-(LED1-Pad2): track 0.00 -> 40.2 mm
- net COL13: track 278.3 -> 318.0 mm
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
Commit message: Remove LED MCU
Parts:
- removed C10, C8, C9: 0.1u, Capacitors_SMD:C_0603
- removed C11, C12, C13, C14: 0.47u, Capacitors_SMD:C_0603
- removed C7: 22u, Capacitors_SMD:C_0805
- removed R2: 100k, Resistors_SMD:R_0603
- removed R8: 20k, Resistors_SMD:R_0603
- removed U4: IS31FL3733, Housings_DFN_QFN:QFN-48-1EP_6x6mm_Pitch0.4mm
Routing:
- net LED-CS1: track 310.3 -> 70.2 mm
- net LED-CS2: track 238.1 -> 0.00 mm, vias 1 -> 0
- net LED-CS3: track 284.3 -> 71.4 mm
- net LED-CS4: track 265.5 -> 72.0 mm
- net LED-CS5: track 249.6 -> 71.9 mm
- net LED-CS6: track 232.5 -> 71.8 mm
- net LED-CS7: track 214.1 -> 71.8 mm
- net LED-CS8: track 196.0 -> 71.8 mm
- net LED-CS9: track 178.0 -> 71.8 mm
- net LED-CS10: track 160.6 -> 71.8 mm
- net GND: track 998.7 -> 914.1 mm, vias 17 -> 10
- net +5V: track 751.8 -> 670.6 mm, vias 24 -> 19
- net LED-CS14: track 101.1 -> 25.7 mm, vias 1 -> 0
- net LED-CS11: track 143.0 -> 71.8 mm
- net LED-SW2: track 262.9 -> 203.8 mm, vias 2 -> 0
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
Commit message: Remove MCU
Parts:
- added C10, C8, C9: 0.1u, Capacitors_SMD:C_0603, B.Cu at (22.1, 117.6)
- added C11, C12, C13, C14: 0.47u, Capacitors_SMD:C_0603, B.Cu at (22.1, 117.6)
- added C7: 22u, Capacitors_SMD:C_0805, B.Cu at (22.1, 117.6)
- added R2: 100k, Resistors_SMD:R_0603, B.Cu at (22.1, 117.6)
- added R8: 20k, Resistors_SMD:R_0603, B.Cu at (22.1, 117.6)
- added U4: IS31FL3733, Housings_DFN_QFN:QFN-48-1EP_6x6mm_Pitch0.4mm, B.Cu at (22.1, 117.6)
- moved R1 75.2 mm to (9.02, 93.4)
- moved C4 74.9 mm to (9.02, 93.4)
- moved C5 71.1 mm to (9.02, 93.4), turned to 0 degrees
- moved U1 68.3 mm to (9.02, 93.4), turned to 0 degrees
- moved C3 67.2 mm to (9.02, 93.4), turned to 0 degrees
- moved C1 63.5 mm to (9.02, 93.4), turned to 0 degrees
- moved C2 61.5 mm to (9.02, 93.4), turned to 0 degrees
- moved U2 60.3 mm to (9.02, 93.4), turned to 0 degrees
- moved C6 60.3 mm to (9.02, 93.4), turned to 0 degrees
Routing:
- net COL15: track 354.9 -> 78.9 mm
- net COL14: track 346.7 -> 94.3 mm
- net COL13: track 318.0 -> 84.3 mm
- net COL12: track 315.5 -> 105.4 mm
- net COL11: track 283.5 -> 84.2 mm
- net COL10: track 271.0 -> 91.2 mm
- net COL9: track 225.4 -> 64.4 mm
- net COL8: track 206.7 -> 64.4 mm
- net COL7: track 188.2 -> 64.3 mm
- net COL6: track 169.9 -> 64.4 mm
- net COL5: track 151.8 -> 64.7 mm
- net COL4: track 133.2 -> 64.4 mm
- net +3V3: track 62.1 -> 0.00 mm, vias 5 -> 0
- net COL3: track 116.3 -> 64.4 mm
- net GND: track 914.1 -> 869.7 mm
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
Commit message: Finish project basic routing
Parts:
- removed SW1: SW_PUSH, Molex-0548190589:PushButton_6x6mm_TH
- SP4: footprint MX_Alps_Hybrid:MX-1.25U -> MX_Alps_Hybrid:MX-1.25U-FLIPPED
- SP6: footprint MX_Alps_Hybrid:MX-6.5U-ReversedStabilizers -> MX_Alps_Hybrid:MX-6.5U-FLIPPED-ReversedStabilizers
- moved REF** 308.4 mm to (55.6, 114.6)
- moved C3 74.3 mm to (83.3, 94.5), turned to 90 degrees
- moved C12 72.8 mm to (94.9, 118.9)
- moved C9 72.8 mm to (94.9, 116.6)
- moved C1 69.6 mm to (76.8, 77.9), turned to 90 degrees
- moved C7 69.3 mm to (91.4, 117.7), turned to 90 degrees
- moved C2 69.2 mm to (77.7, 85.2), turned to 90 degrees
- moved C4 68.8 mm to (77.6, 98.4)
- moved U1 68.3 mm to (77.3, 92.3), turned to 180 degrees
- moved C6 66.8 mm to (75.3, 85.2), turned to 90 degrees
- moved C10 66.7 mm to (87.9, 106.3), turned to 90 degrees
- moved U2 66.2 mm to (73.4, 77.9), turned to 180 degrees
- moved C13 66.1 mm to (88.1, 121.3)
- moved C8 66.1 mm to (88.1, 119.0)
- moved C11 64.5 mm to (85.7, 107.1), turned to 90 degrees
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Connections:
- D66 pad 1: Net-(D66-Pad1) -> ROW4
- D67 pad 1: Net-(D67-Pad1) -> ROW4
- D68 pad 1: Net-(D68-Pad1) -> ROW4
- K_LM1 pad 3: Net-(K_LM1-Pad3) -> LED-CS1
- K_LM1 pad 4: Net-(K_LM1-Pad4) -> LED-SW1
- K_LM2 pad 2: Net-(K_LM2-Pad2) -> Net-(D63-Pad2)
- K_LM2 pad 3: Net-(K_LM2-Pad3) -> LED-CS1
- K_LM2 pad 4: Net-(K_LM2-Pad4) -> LED-SW1
- K_LM3 pad 3: Net-(K_LM3-Pad3) -> LED-CS2
- K_LM3 pad 4: Net-(K_LM3-Pad4) -> LED-SW1
- K_LM4 pad 3: Net-(K_LM4-Pad3) -> LED-CS2
- K_LM4 pad 4: Net-(K_LM4-Pad4) -> LED-SW1
- K_LM5 pad 3: Net-(K_LM5-Pad3) -> LED-CS2
- K_LM5 pad 4: Net-(K_LM5-Pad4) -> LED-SW1
- K_LM6 pad 3: Net-(K_LM6-Pad3) -> LED-CS3
- K_LM6 pad 4: Net-(K_LM6-Pad4) -> LED-SW1
- K_LM7 pad 3: Net-(K_LM7-Pad3) -> LED-CS3
- K_LM7 pad 4: Net-(K_LM7-Pad4) -> LED-SW1
- K_RM1 pad 3: Net-(K_RM1-Pad3) -> LED-CS11
- K_RM1 pad 4: Net-(K_RM1-Pad4) -> LED-SW1
- K_RM2 pad 3: Net-(K_RM2-Pad3) -> LED-CS11
- K_RM2 pad 4: Net-(K_RM2-Pad4) -> LED-SW1
- K_RM3 pad 3: Net-(K_RM3-Pad3) -> LED-CS12
- K_RM3 pad 4: Net-(K_RM3-Pad4) -> LED-SW1
- K_RM4 pad 3: Net-(K_RM4-Pad3) -> LED-CS12
- K_RM4 pad 4: Net-(K_RM4-Pad4) -> LED-SW1
- K_RM5 pad 3: Net-(K_RM5-Pad3) -> LED-CS13
- K_RM5 pad 4: Net-(K_RM5-Pad4) -> LED-SW1
- K_RM6 pad 3: Net-(K_RM6-Pad3) -> LED-CS13
- K_RM6 pad 4: Net-(K_RM6-Pad4) -> LED-SW1
- SP1 pad 1: Net-(SP1-Pad1) -> COL4
- SP1 pad 3: Net-(SP1-Pad3) -> LED-CS5
- SP1 pad 4: Net-(SP1-Pad4) -> LED-SW1
- SP2 pad 1: Net-(SP2-Pad1) -> COL7
- SP2 pad 3: Net-(SP2-Pad3) -> LED-CS8
- SP2 pad 4: Net-(SP2-Pad4) -> LED-SW1
- SP3 pad 1: Net-(SP3-Pad1) -> Net-(D67-Pad2)
- SP3 pad 2: Net-(SP3-Pad2) -> COL7
- SP3 pad 3: Net-(SP3-Pad3) -> LED-CS8
- SP3 pad 4: Net-(SP3-Pad4) -> LED-SW1
- SP4 pad 1: Net-(SP4-Pad1) -> COL7
- SP4 pad 2: Net-(SP4-Pad2) -> Net-(D67-Pad2)
- SP4 pad 3: Net-(SP4-Pad3) -> LED-CS8
- SP4 pad 4: Net-(SP4-Pad4) -> LED-SW1
- SP5 pad 1: Net-(SP5-Pad1) -> COL8
- SP5 pad 3: Net-(SP5-Pad3) -> LED-CS9
- SP5 pad 4: Net-(SP5-Pad4) -> LED-SW1
- SP6 pad 1: Net-(SP6-Pad1) -> Net-(D67-Pad2)
- SP6 pad 2: Net-(SP6-Pad2) -> COL7
- SP6 pad 3: Net-(SP6-Pad3) -> LED-CS8
- SP6 pad 4: Net-(SP6-Pad4) -> LED-SW1
- SP7 pad 1: Net-(SP7-Pad1) -> COL4
- SP7 pad 2: Net-(SP7-Pad2) -> Net-(D66-Pad2)
- SP7 pad 3: Net-(SP7-Pad3) -> LED-CS5
- SP7 pad 4: Net-(SP7-Pad4) -> LED-SW1
- SP8 pad 1: Net-(SP8-Pad1) -> COL7
- SP8 pad 2: Net-(SP8-Pad2) -> Net-(D67-Pad2)
- SP8 pad 3: Net-(SP8-Pad3) -> LED-CS8
- SP8 pad 4: Net-(SP8-Pad4) -> LED-SW1
- SP9 pad 1: Net-(SP9-Pad1) -> COL8
- SP9 pad 2: Net-(SP9-Pad2) -> Net-(D68-Pad2)
- SP9 pad 3: Net-(SP9-Pad3) -> LED-CS9
- SP9 pad 4: Net-(SP9-Pad4) -> LED-SW1
Routing:
- net GND: track 869.7 -> 2038.8 mm, vias 10 -> 73
- net LED-SW1: track 0.00 -> 358.3 mm, vias 0 -> 2
- net LED-CS14: track 25.7 -> 311.2 mm, vias 0 -> 1
- net COL15: track 78.9 -> 354.3 mm
- net LED-CS16: track 86.3 -> 346.7 mm
- net COL14: track 94.3 -> 332.9 mm
- net ROW4: track 77.6 -> 314.0 mm, vias 0 -> 4
- net LED-CS15: track 107.7 -> 337.4 mm
- net LED-CS13: track 88.2 -> 309.0 mm
- net COL13: track 84.3 -> 300.5 mm
- net LED-CS12: track 71.6 -> 281.4 mm
- net COL12: track 105.4 -> 307.4 mm, vias 1 -> 0
- net LED-CS11: track 71.8 -> 262.6 mm
- net COL11: track 84.2 -> 270.2 mm
- net COL10: track 91.2 -> 255.0 mm
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- added copper zone on B.Cu, net GND
Other:
- board size 304.8 x 95.2 mm -> 303.2 x 94.5 mm

Commit message: Tune zones
Parts:
- added SW1: SW_PUSH, Molex-0548190589:PushButton_6x6mm_TH, B.Cu at (54.0, 115.1)
- USB1: footprint Type-C:HRO-TYPE-C-31-M-12-HandSoldering -> Type-C:HRO-TYPE-C-31-M-12
- moved REF** 23.1 mm to (53.2, 137.6)
Routing:
- net GND: track 2038.8 -> 2107.0 mm, vias 73 -> 82
- net PDI_CLK: track 27.4 -> 65.1 mm
- net VCC: track 19.0 -> 23.1 mm
- net Net-(R7-Pad1): track 3.72 -> 5.55 mm
- net COL2: track 113.0 -> 112.1 mm
- net Net-(R6-Pad2): track 3.49 -> 4.28 mm
- net ROW0: track 365.3 -> 365.9 mm
- net D-: track 51.1 -> 50.6 mm
Other:
- board text added: "3V"
- board text removed: "VCC"
