File: Voyager65.sch (KiCad schematic (older format))
At the start: 29 parts, among them P1 TC2030-IDC, SW1 SW_PUSH, U1 ATXMEGA32A4U-AU, U2 MCP1700T-3002E/TT, U3 PRTR5V0U2X, U4 IS31FL3733

Commit message: Replace MCU, route bus
Parts:
- U1: footprint Housings_QFP:TQFP-44_10x10mm_Pitch0.8mm -> Housings_DFN_QFN:QFN-44-1EP_7x7mm_Pitch0.5mm
Connections:
- net COL15: now reaches U1.37 (PR1/XTAL1/TOSC1)
- net LED-CS16: now reaches U4.33 (CS16)
Changed lines of the file:
@@
 F 0 "U1" H 2925 4700 50  0000 L BNN
 F 1 "ATXMEGA32A4U-AU" H 4025 2250 50  0000 L BNN
-F 2 "Housings_QFP:TQFP-44_10x10mm_Pitch0.8mm" H 3675 3500 50  0001 C CIN
+F 2 "Housings_DFN_QFN:QFN-44-1EP_7x7mm_Pitch0.5mm" H 3675 3500 50  0001 C CIN
 F 3 "" H 3675 3500 50  0001 C CNN
 	1    3675 3500
@@
 NoConn ~ 1100 2525
 NoConn ~ 1600 2525
+Text GLabel 7375 5975 0    60   Input ~ 0
+LED-CS16
+Text GLabel 2775 3200 0    60   Input ~ 0
+COL15
 $EndSCHEMATC

Commit message: Tune zones
Parts:
- USB1: footprint Type-C:HRO-TYPE-C-31-M-12-HandSoldering -> Type-C:HRO-TYPE-C-31-M-12
Changed lines of the file:
@@
 F 0 "USB1" H 8025 2175 60  0000 C CNN
 F 1 "HRO-TYPE-C-31-M-12" V 7825 1475 60  0000 C CNN
-F 2 "Type-C:HRO-TYPE-C-31-M-12-HandSoldering" H 8225 1525 60  0001 C CNN
+F 2 "Type-C:HRO-TYPE-C-31-M-12" H 8225 1525 60  0001 C CNN
 F 3 "" H 8225 1525 60  0001 C CNN
 	1    8225 1525

Commit message: Replace reset switch
Parts:
- SW1: footprint Molex-0548190589:PushButton_6x6mm_TH -> Molex-0548190589:SKQG-1155865
Changed lines of the file:
@@
 F 0 "SW1" H 2400 2610 50  0000 C CNN
 F 1 "SW_PUSH" H 2250 2420 50  0000 C CNN
-F 2 "Molex-0548190589:PushButton_6x6mm_TH" H 2250 2500 50  0001 C CNN
+F 2 "Molex-0548190589:SKQG-1155865" H 2250 2500 50  0001 C CNN
 F 3 "" H 2250 2500 50  0000 C CNN
 	1    2250 2500

Commit message: Prepare gerbers for production
Parts:
- removed USB1: HRO-TYPE-C-31-M-12, Type-C:HRO-TYPE-C-31-M-12, symbol HRO-TYPE-C-31-M-12
- added USB1: Wurth-632723300011, Type-C:Wurth-632723300011-MaximumExtensionMount, symbol Wurth-632723300011
Connections:
- net D+: now also USB1.18 (Dp2), USB1.6 (Dp1)
- net D-: now also USB1.19 (Dn2), USB1.7 (Dn1)
- net GND: now also USB1.1 (GND), USB1.12 (GND), USB1.13 (GND), USB1.24 (GND), USB1.25 (Center_Plate_Pin), USB1.26 (Connector_Legs), USB1.27 (Under-Barrel_Pads)
- net VCC: now also USB1.16 (VBUS), USB1.21 (VBUS), USB1.4 (VBUS), USB1.9 (VBUS)
- net at R7.1: now also USB1.17 (CC2)
- net at R6.2: now also USB1.5 (CC1)
- no-connect marks 6 -> 4
Other:
- moved on the sheet: C10, C11, C12, C13, C7, C8, C9, F1, R6, R7, U3

Commit message: Begin fleshing out BOM
Parts:
- U1: value ATXMEGA32A4U-AU -> ATXMEGA32A4U-MH
- U4: value IS31FL3733 -> IS31FL3733-QFLS4-TR
Changed lines of the file:
@@
 P 3675 3500
 F 0 "U1" H 2925 4700 50  0000 L BNN
-F 1 "ATXMEGA32A4U-AU" H 4025 2250 50  0000 L BNN
+F 1 "ATXMEGA32A4U-MH" H 4025 2250 50  0000 L BNN
 F 2 "Housings_DFN_QFN:QFN-44-1EP_7x7mm_Pitch0.5mm" H 3675 3500 50  0001 C CIN
 F 3 "" H 3675 3500 50  0001 C CNN
@@
 P 7875 4475
 F 0 "U4" H 7875 2825 60  0000 C CNN
-F 1 "IS31FL3733" H 7875 5825 60  0000 C CNN
+F 1 "IS31FL3733-QFLS4-TR" H 7875 5825 60  0000 C CNN
 F 2 "Housings_DFN_QFN:QFN-48-1EP_6x6mm_Pitch0.4mm" H 7875 4775 60  0001 C CNN
-F 3 "" H 7875 4775 60  0001 C CNN
+F 3 "http://www.issi.com/WW/pdf/31FL3733.pdf" H 7875 4775 60  0001 C CNN
 	1    7875 4475
 	1    0    0    -1

Commit message: Swap USB back
Parts:
- removed USB1: Wurth-632723300011, Type-C:Wurth-632723300011-MaximumExtensionMount, symbol Wurth-632723300011
- added USB1: HRO-TYPE-C-31-M-12, Type-C:HRO-TYPE-C-31-M-12, symbol HRO-TYPE-C-31-M-12
Connections:
- net D+: now also USB1.6 (DP1), USB1.8 (DP2)
- net D-: now also USB1.5 (DN2), USB1.7 (DN1)
- net GND: now also USB1.1 (GND), USB1.12 (GND), USB1.13 (SHIELD)
- net VCC: now also USB1.11 (VBUS), USB1.2 (VBUS)
- net at R6.2: now also USB1.4 (CC1)
- net at R7.1: now also USB1.10 (CC2)
Other:
- moved on the sheet: F1, R6, R7, U3

Commit message: Remove IS31FL3733
Parts:
- removed C10, C8, C9: 0.1u, Capacitors_SMD:C_0603, symbol C_Small
- removed C11, C12, C13, C14: 0.47u, Capacitors_SMD:C_0603, symbol C_Small
- removed C7: 22u, Capacitors_SMD:C_0805, symbol CP1_Small
- removed R2: 100k, Resistors_SMD:R_0603, symbol R_Small
- removed R3, R4: 1k, Resistors_SMD:R_0603, symbol R_Small
- removed R8: 20k, Resistors_SMD:R_0603, symbol R_Small
- removed U4: IS31FL3733-QFLS4-TR, Housings_DFN_QFN:QFN-48-1EP_6x6mm_Pitch0.4mm, symbol IS31FL3733
Connections:
- net I2C+: no longer names the net of U1.28 (PE0/OC0A/SDA)
- net I2C-: no longer names the net of U1.29 (PE1/OC0B/XCK0/SCL)
- no-connect marks 4 -> 2
